File: hardware/air-ctrl.kicad_pcb (KiCad board)
At the start: 2 copper layers, 75.2 x 35 mm, 67 parts, among them J1 USB_C_Receptacle_USB2.0_16P, J2 SFV24R-2STE1HLF, J3 Conn_ARM_SWD_TagConnect_TC203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, J4 Conn_01x02, Q1 BSS138, SW1 SW_RST, U1 nRF52832-QFxx, U2 BME688, U3 MCP73871-2CC, U4 MCP1700x-330xxTT, U5 USBLC6-2SC6, Y1 32MHz, Y2 32.768kHz

Commit message: wip: layout on the back side
Parts:
- C1, C2, C3, C6, C7, C8, C9, D1, D2, D3, F1, J1, J2, J4, R10, R11, R12, R13, R14, R15, R8, R9, TP1, TP2, TP3, TP4, TP5, TP6, U3, U4, U5: moved to B.Cu
- moved C9 54.3 mm to (154.6, 51.6), turned to 180 degrees
- moved U4 54.0 mm to (154.6, 54.5)
- moved C8 53.6 mm to (155.3, 57.5)
- moved TP3 50.5 mm to (157.9, 57.5)
- moved TP4 47.8 mm to (155.3, 47.9)
- moved C6 47.5 mm to (158.4, 59.9)
- moved U3 45.9 mm to (161.5, 55.6), turned to 0 degrees
- moved R8 41.6 mm to (173.7, 54.2)
- moved TP5 40.6 mm to (151.4, 63.8)
- moved C7 40.5 mm to (155.8, 61.9), turned to 180 degrees
- moved F1 40.2 mm to (173.0, 49.6)
- moved J2 40.2 mm to (170.1, 64.4), turned to 180 degrees
- moved J4 40.2 mm to (154.9, 69.6), turned to 180 degrees
- moved U5 40.2 mm to (173.0, 44.6)
- moved J1 40.2 mm to (181.3, 53.5), turned to -90 degrees
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Routing:
- net /power/V_IN: track 0.00 -> 66.4 mm
- net /power/V_BUS: track 0.00 -> 29.0 mm
- net Net-(U3-THERM): track 0.00 -> 25.2 mm
- net /power/V_3V3: track 28.2 -> 46.8 mm
- net +BATT: track 0.00 -> 18.5 mm
- net Net-(U4-VI): track 0.00 -> 8.88 mm
- net Net-(U3-~{PG}): track 0.45 -> 5.89 mm
- net Net-(U3-STAT2): track 0.00 -> 5.14 mm
- net Net-(U3-STAT1/~{LBO}): track 0.62 -> 5.34 mm
- net Net-(J1-CC1): track 0.00 -> 4.34 mm
- net Net-(U3-PROG1): track 0.00 -> 4.32 mm
- net Net-(U3-PROG3): track 0.00 -> 3.77 mm
- net -BATT: track 35.7 -> 38.6 mm
- net Net-(J1-CC2): track 0.00 -> 2.73 mm
- net Net-(U5-GND): track 0.00 -> 2.50 mm
Other:
- board size 75.2 x 35 mm -> 35 x 35 mm

Commit message: connected power and signals, gnd missing
Parts:
- moved TP7 4.99 mm to (162.5, 41.1)
- moved R2 3.69 mm to (162.9, 71.3)
- moved R1 3.51 mm to (161.3, 71.3)
- moved L1 2.01 mm to (175.6, 58.3)
- moved TP8 1.93 mm to (161.5, 43.1)
- moved C12 0.58 mm to (170.3, 56.9)
- moved C10 0.55 mm to (170.3, 58.4)
- moved J3 0.55 mm to (173.3, 71.2)
- moved C15 0.42 mm to (152.6, 59.1)
- moved C16 0.42 mm to (152.6, 60.6)
- moved Y2 0.42 mm to (155.5, 59.8)
Routing:
- net /power/V_3V3: track 46.8 -> 147.5 mm, vias 0 -> 3
- net Net-(J3-SWDIO): track 14.8 -> 39.1 mm, vias 0 -> 2
- net /display/LEDK: track 0.00 -> 22.7 mm, vias 0 -> 1
- net /display/DISP_RST: track 5.61 -> 25.2 mm, vias 0 -> 1
- net /mcu/I2C_SCL: track 13.8 -> 32.2 mm, vias 0 -> 2
- net /display/DISP_SCLK: track 0.00 -> 18.1 mm, vias 0 -> 1
- net /display/DISP_CS: track 6.48 -> 23.2 mm, vias 0 -> 1
- net /display/DISP_DC: track 0.00 -> 15.8 mm, vias 0 -> 1
- net /display/DISP_MOSI: track 0.00 -> 14.6 mm, vias 0 -> 1
- net Net-(J3-SWCLK): track 28.8 -> 25.7 mm
- net /mcu/I2C_SDA: track 17.4 -> 19.9 mm
- net Net-(U1-ANT): track 12.1 -> 10.2 mm
- net Net-(U1-P0.01/XL2): track 9.42 -> 8.67 mm
- net Net-(J3-~{RESET}): track 22.9 -> 23.5 mm
- net Net-(J3-SWO): track 33.6 -> 34.2 mm

Commit message: wip layout
Parts:
- moved L1 4.17 mm to (176.7, 54.2)
- moved R16 3.93 mm to (180.1, 53.4)
- moved C17 3.93 mm to (182.4, 52.6)
- moved C19 3.93 mm to (182.4, 54.1)
- moved TP7 3.64 mm to (165.1, 43.7)
Routing:
- net /power/V_3V3: track 147.5 -> 170.2 mm
- net -BATT: track 38.7 -> 34.5 mm
- net Net-(AE1-A): track 12.7 -> 8.55 mm
- net Net-(U1-ANT): track 10.2 -> 14.2 mm
- net Net-(U4-VI): track 8.88 -> 10.0 mm
- net /mcu/I2C_SCL: track 32.2 -> 31.4 mm
- net Net-(C19-Pad1): track 3.49 -> 4.21 mm
Changed lines of the file:
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@@
 		(tags "resistor")
 		(property "Reference" "R7"
-			(at -2.125 3.34 90)
+			(at -1.055 1.66 180)
 			(layer "F.SilkS")
 			(effects
@@
 	(footprint "Capacitor_SMD:C_0603_1608Metric"
 		(layer "F.Cu")
-		(at 180.305 57.44)
+		(at 182.365 54.09)
 		(descr "Capacitor SMD 0603 (1608 Metric), square (rectangular) end terminal, IPC-7351 nominal, (Body size source: IPC-SM-782 page 76, https://www.pcb-3d.com/wordpress/wp-content/uploads/ipc-sm-782a_amendment_1_and_2.pdf), generated with kicad-footprint-generator")
 		(tags "capacitor")
@@
 		(tags "inductor")
 		(property "Reference" "L2"
-			(at -2.7625 0.16 90)
+			(at -0.8525 1.72 180)
 			(layer "F.SilkS")
 			(effects
@@
 	(footprint "Resistor_SMD:R_0603_1608Metric"
 		(layer "F.Cu")
-		(at 178.03 56.765 -90)
+		(at 180.09 53.415 -90)
 		(descr "Resistor SMD 0603 (1608 Metric), square (rectangular) end terminal, IPC-7351 nominal, (Body size source: IPC-SM-782 page 72, https://www.pcb-3d.com/wordpress/wp-content/uploads/ipc-sm-782a_amendment_1_and_2.pdf), generated with kicad-footprint-generator")
 		(tags "resistor")
@@
 		(at 155.2 42.5)
 		(property "Reference" "U2"
-			(at 8.64 3.45 270)
+			(at 1.45 2.41 0)
 			(layer "F.SilkS")
 			(effects
@@
 		(tags "resistor")
 		(property "Reference" "R6"
-			(at 0.675 -2 180)
+			(at -1.315 -1.62 180)
 			(layer "F.SilkS")
 			(effects
@@
 	(footprint "Inductor_SMD:L_0603_1608Metric"
 		(layer "F.Cu")
-		(at 175.5975 58.28 180)
+		(at 176.6625 54.25 180)
 		(descr "Inductor SMD 0603 (1608 Metric), square (rectangular) end terminal, IPC-7351 nominal, (Body size source: http://www.tortai-tech.com/upload/download/2011102023233369053.pdf), generated with kicad-footprint-generator")
 		(tags "inductor")
@@
 		(tags "capacitor")
 		(property "Reference" "C5"
-			(at 8.065 -4.55 90)
+			(at 2.425 -0.31 180)
 			(layer "F.SilkS")
 			(effects
@@
 	(footprint "Capacitor_SMD:C_0603_1608Metric"
 		(layer "F.Cu")
-		(at 180.305 55.94)
+		(at 182.365 52.59)
 		(descr "Capacitor SMD 0603 (1608 Metric), square (rectangular) end terminal, IPC-7351 nominal, (Body size source: IPC-SM-782 page 76, https://www.pcb-3d.com/wordpress/wp-content/uploads/ipc-sm-782a_amendment_1_and_2.pdf), generated with kicad-footprint-generator")
 		(tags "capacitor")
@@
 	(footprint "TestPoint:TestPoint_Pad_D1.0mm"
 		(layer "F.Cu")
-		(at 162.52 41.12)
+		(at 165.1 43.69)
 		(descr "SMD pad as test Point, diameter 1.0mm")
 		(tags "test point SMD pad")
 		(property "Reference" "TP7"
-			(at -13.43 9.765 0)
+			(at 0.58 1.73 0)
 			(layer "F.SilkS")
 			(effects
@@
 	)
 	(segment
-		(start 179.58 55.89)
-		(end 179.53 55.94)
+		(start 181.64 52.54)
+		(end 181.59 52.59)
 		(width 0.2)
 		(layer "F.Cu")
@@
 	)
 	(segment
-		(start 179.53 55.94)
-		(end 179.53 47.645)
+		(start 180.09 52.59)
+		(end 181.59 52.59)
 		(width 0.2)
 		(layer "F.Cu")
@@
 	)
 	(segment
-		(start 178.03 55.94)
-		(end 179.53 55.94)
+		(start 181.59 52.59)
+		(end 181.59 45.665)
 		(width 0.2)
 		(layer "F.Cu")
@@
 	)
 	(segment
-		(start 179.53 47.645)
+		(start 181.59 45.665)
 		(end 181.55 45.625)
 		(width 0.2)
@@
 	)
 	(segment
-		(start 181.08 55.94)
-		(end 181.08 48.195)
-		(width 0.2)
-		(layer "F.Cu")
-		(net 2)
-	)
-	(segment
 		(start 153.05 45.5)
 		(end 153.05 45.05)
@@
 	)
 	(segment
-		(start 181.08 48.195)
-		(end 183.65 45.625)
+		(start 169.25 54.015)
+		(end 169.4 53.865)
 		(width 0.2)
 		(layer "F.Cu")
@@
 	)
 	(segment
-		(start 169.25 54.015)
-		(end 169.4 53.865)
+		(start 183.14 52.59)
+		(end 183.14 46.135)
 		(width 0.2)
 		(layer "F.Cu")
@@
 	)
 	(segment
-		(start 181.08 55.94)
-		(end 181.08 57.44)
+		(start 183.14 52.59)
+		(end 183.14 54.09)
 		(width 0.2)
 		(layer "F.Cu")
@@
 	)
 	(segment
+		(start 183.14 46.135)
+		(end 183.65 45.625)
+		(width 0.2)
+		(layer "F.Cu")
+		(net 2)
+	)
+	(segment
 		(start 153.05 45.05)
 		(end 154 44.1)
@@
 	)
 	(segment
+		(start 164.7 41.5)
+		(end 166.95 43.75)
+		(width 0.2)
+		(layer "F.Cu")
+		(net 3)
+	)
+	(segment
 		(start 153 50.61)
 		(end 150.78 52.83)
@@
 	)
 	(segment
+		(start 166.95 49.19)
+		(end 164.98 51.16)
+		(width 0.2)
+		(layer "F.Cu")
+		(net 3)
+	)
+	(segment
 		(start 158.4 42.1)
 		(end 159 41.5)
@@
 	)
 	(segment
+		(start 164.98 51.16)
+		(end 164.98 56.77)
+		(width 0.2)
+		(layer "F.Cu")
+		(net 3)
+	)
+	(segment
 		(start 153.79 49.82)
 		(end 151.5 47.53)
@@
 	)
 	(segment
+		(start 159 41.5)
+		(end 164.7 41.5)
+		(width 0.2)
+		(layer "F.Cu")
+		(net 3)
+	)
+	(segment
 		(start 153.625 42.9)
 		(end 154 42.9)
@@
 	)
 	(segment
+		(start 166.95 43.75)
+		(end 166.95 49.19)
+		(width 0.2)
+		(layer "F.Cu")
+		(net 3)
+	)
+	(segment
 		(start 159.83 61.92)
 		(end 159.83 72.16)
@@
 	)
 	(segment
-		(start 161.5 58.5)
-		(end 161.34 58.66)
-		(width 0.2)
-		(layer "B.Cu")
-		(net 4)
-	)
-	(segment
 		(start 156.5575 53.5275)
 		(end 156.5575 44.1575)
@@
 	)
 	(segment
-		(start 160.34 42.575)
-		(end 162.54 42.575)
+		(start 162 58)
+		(end 162 57.5375)
 		(width 0.2)
 		(layer "B.Cu")
@@
 	)
 	(segment
-		(start 162 58)
-		(end 161.34 58.66)
+		(start 160.34 42.575)
+		(end 162.54 42.575)
 		(width 0.2)
 		(layer "B.Cu")
@@
 	)
 	(segment
-		(start 162 57.5375)
+		(start 161.34 58.66)
 		(end 162 58)
 		(width 0.2)
@@
 	)
 	(segment
+		(start 157.87 57.55)
+		(end 157.87 57.045)
+		(width 0.2)
+		(layer "B.Cu")
+		(net 6)
+	)
+	(segment
 		(start 157.185 55.47)
 		(end 154.55 55.47)
@@
 	)
 	(segment
+		(start 157.87 57.045)
+		(end 158.315 56.6)
+		(width 0.2)
+		(layer "B.Cu")
+		(net 6)
+	)
+	(segment
 		(start 169.53 58.37)
 		(end 169.55 58.39)
@@
 	)
 	(segment
-		(start 177.34 58.28)
-		(end 178.03 57.59)
+		(start 180.09 54.24)
+		(end 177.46 54.24)
 		(width 0.2)
 		(layer "F.Cu")
@@
 	)
 	(segment
-		(start 179.53 57.44)
-		(end 178.18 57.44)
+		(start 181.59 54.09)
+		(end 180.24 54.09)
 		(width 0.2)
 		(layer "F.Cu")
@@
 	)
 	(segment
-		(start 176.385 58.28)
-		(end 177.34 58.28)
+		(start 180.24 54.09)
+		(end 180.09 54.24)
 		(width 0.2)
 		(layer "F.Cu")
@@
 	)
 	(segment
-		(start 178.18 57.44)
-		(end 178.03 57.59)
+		(start 177.46 54.24)
+		(end 177.45 54.25)
 		(width 0.2)
 		(layer "F.Cu")
@@
 	(segment
 		(start 173.06 59.17)
-		(end 173.95 58.28)
+		(end 175.875 56.355)
 		(width 0.2)
 		(layer "F.Cu")
@@
 	)
 	(segment
-		(start 164.98 59.17)
-		(end 173.06 59.17)
+		(start 175.875 56.355)
+		(end 175.875 54.25)
 		(width 0.2)
 		(layer "F.Cu")
@@
 	)
 	(segment
-		(start 173.95 58.28)
-		(end 174.81 58.28)
+		(start 164.98 59.17)
+		(end 173.06 59.17)
 		(width 0.2)
 		(layer "F.Cu")
@@
 	)
 	(segment
-		(start 163.83 41.41)
-		(end 164.09 41.15)
+		(start 165.1 42.82)
+		(end 164.72 42.44)
 		(width 0.2)
 		(layer "F.Cu")
@@
 	)
 	(segment
-		(start 164.09 41.15)
-		(end 162.55 41.15)
+		(start 157.2 43.7)
+		(end 158 44.5)
 		(width 0.2)
 		(layer "F.Cu")
@@
 	)
 	(segment
-		(start 163.83 56.02)
-		(end 163.83 46.33)
+		(start 156.4 43.7)
+		(end 157.2 43.7)
 		(width 0.2)
 		(layer "F.Cu")
@@
 	)
 	(segment
-		(start 162.55 41.15)
-		(end 162.52 41.12)
+		(start 164.72 42.44)
+		(end 164.2 42.44)
 		(width 0.2)
 		(layer "F.Cu")
@@
 	)
 	(segment
-		(start 157.2 43.7)
-		(end 158 44.5)
+		(start 163.83 42.81)
+		(end 164.2 42.44)
 		(width 0.2)
 		(layer "F.Cu")
@@
 	)
 	(segment
-		(start 156.4 43.7)
-		(end 157.2 43.7)
+		(start 165.1 43.69)
+		(end 165.1 42.82)
 		(width 0.2)
 		(layer "F.Cu")
@@
 	)
 	(segment
-		(start 158 44.5)
-		(end 159 44.5)
+		(start 163.83 56.02)
+		(end 163.83 42.81)
 		(width 0.2)
 		(layer "F.Cu")
@@
 	)
 	(segment
-		(start 155.02 44.76)
-		(end 155.34 44.76)
+		(start 158 44.5)
+		(end 159 44.5)
 		(width 0.2)
 		(layer "F.Cu")
@@
 	)
 	(segment
-		(start 163.83 46.33)
-		(end 163.83 41.41)
+		(start 155.02 44.76)
+		(end 155.34 44.76)
 		(width 0.2)
 		(layer "F.Cu")
@@
 	)
 	(via
-		(at 164.09 41.15)
+		(at 164.2 42.44)
 		(size 0.6)
 		(drill 0.3)
@@
 	)
 	(segment
-		(start 164.09 41.15)
-		(end 158.087854 41.15)
+		(start 163.5465 41.7865)
+		(end 164.2 42.44)
+		(width 0.2)
+		(layer "B.Cu")
+		(net 47)
+	)
+	(segment
+		(start 157.451354 41.7865)
+		(end 163.5465 41.7865)
 		(width 0.2)
 		(layer "B.Cu")
@@
 	)
 	(segment
-		(start 158.087854 41.15)
-		(end 155.02 44.217854)
+		(start 155.02 44.217854)
+		(end 157.451354 41.7865)
 		(width 0.2)
 		(layer "B.Cu")

Commit message: fixed connections to ground and DRC
Parts:
- moved R11 2.29 mm to (167.1, 52.9)
- moved C12 1.16 mm to (171.3, 56.2)
- moved C10 0.81 mm to (170.7, 57.7)
- turned C8 to 180 degrees
Routing:
- net -BATT: track 34.5 -> 76.3 mm, vias 0 -> 26
- net Net-(U1-DEC3): track 5.03 -> 6.26 mm
- net Net-(U3-THERM): track 25.2 -> 24.1 mm
- net Net-(U4-VI): track 10.0 -> 10.7 mm
- net Net-(U1-DEC2): track 4.58 -> 5.21 mm
- added copper zone on B.Cu, net -BATT
- added copper zone on F.Cu, net -BATT
