File: hardware/air-ctrl.kicad_pcb (KiCad board)
At the start: 2 copper layers, 35 x 35 mm, 67 parts, among them J1 USB_C_Receptacle_USB2.0_16P, J2 SFV24R-2STE1HLF, J3 Conn_ARM_SWD_TagConnect_TC203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, J4 Conn_01x02, Q1 BSS138, SW1 SW_RST, U1 nRF52832-QFxx, U2 BME688, U3 MCP73871-2CC, U4 MCP1700x-330xxTT, U5 USBLC6-2SC6, Y1 32MHz, Y2 32.768kHz

Commit message: fixed antenna layout
wip: placing components
Parts:
- removed U5: USBLC6-2SC6, Package_TO_SOT_SMD:SOT-23-6
- added C24: 100nF, Capacitor_SMD:C_0603_1608Metric, B.Cu at (170.3, 44.5)
- added C25: 0.8pF, Capacitor_SMD:C_0201_0603Metric, F.Cu at (163.1, 49.9)
- added C26: NC, Capacitor_SMD:C_0201_0603Metric, F.Cu at (161.0, 50.1)
- added D4: ESD5Zxx, Diode_SMD:D_SOD-523, B.Cu at (173.6, 44.7)
- AE1: value BLE -> ~; footprint RF_Antenna:Texas_SWRA117D_2.4GHz_Left -> RF_Antenna:Antenna_BLE
- C17: value 0.8pF -> 1.5pF; footprint Capacitor_SMD:C_0603_1608Metric -> Capacitor_SMD:C_0201_0603Metric
- C19: value 0.8pF -> 0.5pF; footprint Capacitor_SMD:C_0603_1608Metric -> Capacitor_SMD:C_0201_0603Metric
- L1: value 3.9nH -> 4.7nH; footprint Inductor_SMD:L_0603_1608Metric -> Inductor_SMD:L_0201_0603Metric
- R16: footprint Resistor_SMD:R_0603_1608Metric -> Resistor_SMD:R_0201_0603Metric
- Y2: footprint Crystal:Crystal_SMD_2016-4Pin_2.0x1.6mm -> Crystal:Crystal_SMD_3215-2Pin_3.2x1.5mm
- moved R1 37.9 mm to (176.4, 36.5), turned to -90 degrees
- moved R2 36.8 mm to (174.9, 36.5), turned to -90 degrees
- moved J3 30.8 mm to (158.6, 44.1), turned to 90 degrees
- moved Q1 30.2 mm to (180.6, 46.9), turned to 0 degrees
- moved R5 30.0 mm to (180.2, 44.4), turned to 180 degrees
- moved U2 29.4 mm to (158.5, 71.7), turned to 90 degrees
- moved C4 29.2 mm to (162.6, 72.8), turned to 90 degrees
- moved C5 28.5 mm to (164.2, 72.8), turned to 90 degrees
- moved AE1 28.1 mm to (153.7, 48.8), turned to 90 degrees
- moved C17 26.5 mm to (155.9, 53.3), turned to 90 degrees
- moved TP8 25.1 mm to (156.5, 67.7), turned to 90 degrees
- moved C16 24.9 mm to (175.6, 50.9), turned to 0 degrees
- moved SW1 24.7 mm to (164.2, 42.4), turned to -90 degrees
- moved C19 24.3 mm to (158.1, 53.2), turned to 90 degrees
- moved R6 24.2 mm to (159.8, 66.5), turned to 0 degrees
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Connections:
- C23 pad 1: Net-(C23-Pad1) -> -BATT
- C23 pad 2: -BATT -> Net-(J3-~{RESET})
- F1 pad 1: Net-(U5-GND) -> /power/V_BUS
- SW1 pad 1: Net-(C23-Pad1) -> -BATT
Routing:
- net /power/V_3V3: track 170.2 -> 0.00 mm, vias 3 -> 0
- net -BATT: track 76.3 -> 0.00 mm, vias 26 -> 0
- net /power/V_IN: track 66.2 -> 0.00 mm
- net Net-(J3-SWDIO): track 39.2 -> 0.00 mm, vias 2 -> 0
- net Net-(J3-SWO): track 34.2 -> 0.00 mm
- net /mcu/I2C_SCL: track 31.4 -> 0.00 mm, vias 2 -> 0
- net /power/V_BUS: track 29.0 -> 0.00 mm
- net Net-(J3-SWCLK): track 25.7 -> 0.00 mm
- net /display/DISP_RST: track 25.2 -> 0.00 mm, vias 1 -> 0
- net Net-(U3-THERM): track 24.1 -> 0.00 mm
- net Net-(J3-~{RESET}): track 23.5 -> 0.00 mm
- net /display/DISP_CS: track 23.2 -> 0.00 mm, vias 1 -> 0
- net /display/LEDK: track 22.7 -> 0.00 mm, vias 1 -> 0
- net /mcu/I2C_SDA: track 19.9 -> 0.00 mm
- net +BATT: track 18.5 -> 0.00 mm
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- removed copper zone on B.Cu, net -BATT
- removed copper zone on F.Cu, net -BATT

Commit message: Fixed layout bottom layer
Also fixed all DRC issues
Parts:
- C7: value 10uF -> 4.7uF
- moved TP6 35.7 mm to (159.8, 73.5)
- moved D4 30.2 mm to (157.6, 70.3), turned to -90 degrees
- moved C24 28.3 mm to (159.1, 70.5), turned to -90 degrees
- moved J4 25.4 mm to (180.3, 69.8)
- moved TP4 25.2 mm to (155.9, 73.0)
- moved TP1 24.8 mm to (183.8, 64.0)
- moved TP5 24.4 mm to (175.8, 64.9)
- moved J1 22.4 mm to (167.7, 71.3), turned to 180 degrees
- moved F1 22.0 mm to (158.6, 66.2), turned to 0 degrees
- moved C1 20.2 mm to (178.8, 45.5), turned to -90 degrees
- moved C2 18.1 mm to (180.3, 45.5), turned to -90 degrees
- moved C3 16.1 mm to (181.8, 45.5), turned to -90 degrees
- moved R9 13.5 mm to (166.5, 65.2), turned to 0 degrees
- moved C7 13.3 mm to (169.1, 62.7), turned to -90 degrees
- moved J2 13.3 mm to (174.2, 51.8), turned to -90 degrees
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Routing:
- net /power/V_3V3: track 0.00 -> 45.6 mm
- net -BATT: track 0.00 -> 27.2 mm
- net /mcu/I2C_SDA: track 0.00 -> 26.2 mm
- net +BATT: track 0.00 -> 23.6 mm
- net /power/V_BUS: track 0.00 -> 23.2 mm
- net Net-(J3-SWO): track 0.00 -> 22.4 mm
- net /mcu/I2C_SCL: track 0.00 -> 22.2 mm
- net /power/V_IN: track 0.00 -> 21.9 mm, vias 0 -> 2
- net /display/DISP_DC: track 0.00 -> 16.0 mm, vias 0 -> 1
- net /display/DISP_RST: track 0.00 -> 13.3 mm, vias 0 -> 1
- net /display/DISP_CS: track 0.00 -> 13.2 mm, vias 0 -> 1
- net Net-(U1-XC1): track 0.00 -> 12.7 mm
- net /display/DISP_BL: track 0.00 -> 12.4 mm
- net /display/DISP_MOSI: track 0.00 -> 12.0 mm, vias 0 -> 1
- net Net-(J3-~{RESET}): track 0.00 -> 11.6 mm
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
Commit message: routing power lines, fixing schematic
using 3.3V to power LEDs, fixed  CE-pin to be low
Parts:
- moved TP1 2.66 mm to (181.3, 63.1)
- moved TP7 0.78 mm to (159.8, 64.4)
- moved R6 0.76 mm to (162.6, 69.1), turned to 180 degrees
- moved TP4 0.54 mm to (155.8, 73.6)
- moved TP6 0.45 mm to (159.7, 73.0)
Connections:
- D1 pad 2: /power/V_IN -> /power/V_3V3
- D2 pad 2: /power/V_IN -> /power/V_3V3
- D3 pad 2: /power/V_IN -> /power/V_3V3
- U3 pad 9: Net-(U3-THERM) -> -BATT
Routing:
- net /power/V_3V3: track 45.6 -> 190.2 mm, vias 0 -> 9
- net /display/LEDK: track 0.00 -> 9.83 mm, vias 0 -> 1
- net -BATT: track 27.2 -> 21.2 mm
- net /power/V_IN: track 21.9 -> 17.5 mm
- net +BATT: track 23.6 -> 21.1 mm
- net /mcu/I2C_SCL: track 22.2 -> 23.5 mm

Commit message: improved layout to shorten 3.3V power traces
Parts:
- C8, C9, TP3, TP4, U4: moved to F.Cu
- moved TP4 27.6 mm to (181.3, 63.0), turned to 90 degrees
- moved TP3 26.2 mm to (183.3, 59.4), turned to 90 degrees
- moved C8 22.9 mm to (181.7, 57.2), turned to 0 degrees
- moved U2 22.2 mm to (180.7, 71.7), turned to 180 degrees
- moved U4 22.1 mm to (179.5, 58.9), turned to 90 degrees
- moved C9 20.8 mm to (177.1, 60.0), turned to 90 degrees
- moved C4 20.5 mm to (182.2, 66.5), turned to 0 degrees
- moved C5 18.6 mm to (182.2, 68.1), turned to 0 degrees
- moved TP8 16.4 mm to (173.0, 63.2), turned to 180 degrees
- moved R6 8.67 mm to (168.6, 62.8)
- moved TP7 7.50 mm to (166.5, 67.8), turned to 180 degrees
- moved R5 6.99 mm to (176.6, 48.4), turned to -90 degrees
- moved R7 6.13 mm to (165.6, 65.0)
- moved Q1 3.67 mm to (179.1, 48.0), turned to 90 degrees
- moved C19 0.09 mm to (158.1, 53.2)
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Routing:
- net Net-(U4-VI): track 10.9 -> 53.8 mm, vias 0 -> 3
- net /power/V_3V3: track 190.2 -> 153.4 mm, vias 9 -> 6
- net /mcu/I2C_SCL: track 23.5 -> 30.7 mm
- net -BATT: track 21.2 -> 14.9 mm
- net /display/DISP_BL: track 12.4 -> 8.89 mm
- net /display/LEDK: track 9.83 -> 7.56 mm
- net /mcu/I2C_SDA: track 26.7 -> 28.8 mm

Commit message: Added name and revision
Parts:
- added TP9: TP_GND, TestPoint:TestPoint_Pad_D1.0mm, F.Cu at (159.2, 72.1)
Other:
- board text added: "${NAME}-${REVISION}"
Changed lines of the file:
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@@
 	)
 	(paper "A4")
+	(title_block
+		(title "air-ctrl")
+		(date "2025-10-18")
+		(rev "1.1")
+	)
 	(layers
 		(0 "F.Cu" signal)
@@
 		)
 	)
+	(property "NAME" "air-ctrl")
 	(net 0 "")
 	(net 1 "Net-(AE1-FEED)")
@@
 		)
 	)
+	(footprint "TestPoint:TestPoint_Pad_D1.0mm"
+		(layer "F.Cu")
+		(at 159.18 72.07)
+		(descr "SMD pad as test Point, diameter 1.0mm")
+		(tags "test point SMD pad")
+		(property "Reference" "TP9"
+			(at 0 -1.448 0)
+			(layer "F.SilkS")
+			(effects
+				(font
+					(size 1 1)
+					(thickness 0.15)
+				)
+			)
+		)
+		(property "Value" "TP_GND"
+			(at 0 1.55 0)
+			(layer "F.Fab")
+			(effects
+				(font
+					(size 1 1)
+					(thickness 0.15)
+				)
+			)
+		)
+		(property "Datasheet" "~"
+			(at 0 0 0)
+			(unlocked yes)
+			(layer "F.Fab")
+			(hide yes)
+			(effects
+				(font
+					(size 1.27 1.27)
+					(thickness 0.15)
+				)
+			)
+		)
+		(property "Description" "test point"
+			(at 0 0 0)
+			(unlocked yes)
+			(layer "F.Fab")
+			(hide yes)
+			(effects
+				(font
+					(size 1.27 1.27)
+					(thickness 0.15)
+				)
+			)
+		)
+		(property ki_fp_filters "Pin* Test*")
+		(sheetname "/power/")
+		(sheetfile "power.kicad_sch")
+		(attr exclude_from_pos_files)
+		(fp_circle
+			(center 0 0)
+			(end 0 0.7)
+			(stroke
+				(width 0.12)
+				(type solid)
+			)
+			(fill no)
+			(layer "F.SilkS")
+		)
+		(fp_circle
+			(center 0 0)
+			(end 1 0)
+			(stroke
+				(width 0.05)
+				(type solid)
+			)
+			(fill no)
+			(layer "F.CrtYd")
+		)
+		(fp_text user "${REFERENCE}"
+			(at 0 -1.45 0)
+			(layer "F.Fab")
+			(effects
+				(font
+					(size 1 1)
+					(thickness 0.15)
+				)
+			)
+		)
+		(pad "1" smd circle
+			(at 0 0)
+			(size 1 1)
+			(layers "F.Cu" "F.Mask")
+			(net 2 "-BATT")
+			(pinfunction "1")
+			(pintype "passive")
+		)
+		(embedded_fonts no)
+	)
 	(footprint "Capacitor_SMD:C_0201_0603Metric"
 		(layer "F.Cu")
@@
 		)
 	)
+	(gr_text "${NAME}-${REVISION}"
+		(at 152.82 74.75 90)
+		(layer "F.SilkS")
+		(effects
+			(font
+				(size 1.5 1.5)
+				(thickness 0.3)
+				(bold yes)
+			)
+			(justify left bottom)
+		)
+	)

Commit message: Fixed DRC issues on antenna pad and trace
Parts:
- moved AE1 0.09 mm to (153.7, 48.9)
Changed lines of the file:
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@@
 	(footprint "RF_Antenna:Antenna_BLE"
 		(layer "F.Cu")
-		(at 153.6565 48.81 90)
+		(at 153.71 48.88 90)
 		(property "Reference" "AE1"
 			(at 7.17 -0.9165 0)
@@
 		(net_tie_pad_groups "1")
 		(fp_line
-			(start 5.29 -2.98)
-			(end 5.29 -0.02)
+			(start 5.380104 -3.04)
+			(end 5.380104 -0.08)
 			(stroke
 				(width 0.254)
@@
 		)
 		(fp_line
-			(start 3.41 -2.98)
-			(end 5.29 -2.98)
+			(start 3.500104 -3.04)
+			(end 5.380104 -3.04)
 			(stroke
 				(width 0.254)
@@
 		)
 		(fp_line
-			(start 1.46 -2.98)
-			(end 1.46 -0.04)
+			(start 1.550104 -3.04)
+			(end 1.550104 -0.1)
 			(stroke
 				(width 0.254)
@@
 		)
 		(fp_line
-			(start -0.52 -2.98)
-			(end 1.46 -2.98)
+			(start -0.429896 -3.04)
+			(end 1.550104 -3.04)
 			(stroke
 				(width 0.254)
@@
 		)
 		(fp_line
-			(start -2.57 -2.94)
-			(end -2.57 0)
+			(start -2.479896 -3)
+			(end -2.479896 -0.06)
 			(stroke
 				(width 0.254)
@@
 		)
 		(fp_line
-			(start -4.79 -2.94)
-			(end -2.57 -2.94)
+			(start -4.699896 -3)
+			(end -2.479896 -3)
 			(stroke
 				(width 0.254)
@@
 		)
 		(fp_line
-			(start 3.41 -0.04)
-			(end 3.41 -2.98)
+			(start 3.500104 -0.1)
+			(end 3.500104 -3.04)
 			(stroke
 				(width 0.254)
@@
 		)
 		(fp_line
-			(start 1.46 -0.04)
-			(end 3.41 -0.04)
+			(start 1.550104 -0.1)
+			(end 3.500104 -0.1)
 			(stroke
 				(width 0.254)
@@
 		)
 		(fp_line
-			(start -0.52 0)
-			(end -0.52 -2.98)
+			(start -0.429896 -0.06)
+			(end -0.429896 -3.04)
 			(stroke
 				(width 0.254)
@@
 		)
 		(fp_line
-			(start -2.57 0)
-			(end -0.52 0)
+			(start -2.479896 -0.06)
+			(end -0.429896 -0.06)
 			(stroke
 				(width 0.254)
@@
 		)
 		(fp_line
-			(start -4.8 1.7)
-			(end -4.790104 -2.94)
+			(start -4.709896 1.64)
+			(end -4.7 -3)
 			(stroke
 				(width 0.254)
@@
 		)
 		(pad "1" connect roundrect
-			(at -4.8 1.85 180)
+			(at -4.709896 1.79 180)
 			(size 0.377 0.254)
 			(layers "F.Cu" "F.Mask")
@@
 		)
 		(group ""
-			(members "209a0455-04f6-4b58-b0ae-014dd7f7e8bc" "2509789c-07dd-4dd8-a51f-43c243804211"
-				"26a550a0-0e9e-42ae-ae6a-5513f2a037a7" "2a4eed77-9d9f-4b0f-ba56-ba25d8e712e8"
-				"4f7e4597-fbac-4e23-aed2-afa333fae4f6" "55c94455-214e-4ffb-a6da-015bdf38ccf6"
-				"705c0e73-2bbe-4a66-b21e-bebf5369d946" "994df067-cb94-43e8-8fc0-f8c08f739cad"
-				"d8a0ef51-1bcc-4bfa-a21e-0bc05fa7d346" "e0c5d7c5-d813-4090-9b40-0154119800ae"
-				"e7c0935a-e132-4bfe-911e-57bb95cab03a" "ff8d8c75-0cb4-45cd-b153-e8660f922aba"
+			(members "28919dec-981b-449c-8571-14b3c1193a38" "36499084-ff91-43a0-9559-5762354c162e"
+				"40a73ee6-07f7-4537-9c1d-6c57c1513f92" "5895e3f0-3bd3-41a0-b642-3b390754c57b"
+				"62b5ca1d-d3de-4e46-8a23-bc883b20b2ab" "6c8e7c77-08ca-4a85-ba5d-5a3286ddfb7c"
+				"75b1eca4-620c-4eff-8bdc-2bc21a9c6d79" "8d3f4351-a146-4af2-b67d-fe788fbdf3c5"
+				"afcf701b-003e-42b7-b24e-b941a6066965" "b3a84e2a-ce09-4ddf-ade8-84811e1e0511"
+				"c99fd7f9-daf0-4e98-9e11-d4545e4ea354" "e7c0935a-e132-4bfe-911e-57bb95cab03a"
 			)
 		)
@@
 	)
 	(segment
-		(start 155.5065 53.61)
-		(end 155.9 53.61)
+		(start 155.678274 53.59)
+		(end 155.677999 53.590275)
 		(width 0.2)
 		(layer "F.Cu")
@@
 	)
 	(segment
+		(start 155.92 53.59)
+		(end 155.678274 53.59)
+		(width 0.2)
+		(layer "F.Cu")
+		(net 1)
+	)
+	(segment
 		(start 156.675 53.59)
 		(end 156.705 53.62)
@@
 		(polygon
 			(pts
-				(xy 149.95 39.85) (xy 149.95 54.8) (xy 155.35 54.8) (xy 155.35 39.86)
+				(xy 149.95 39.85) (xy 149.95 54.8) (xy 155.35 54.8) (xy 155.35 53.91) (xy 155.2 53.91) (xy 155.2 53.3)
+				(xy 155.35 53.3) (xy 155.35 39.86)
 			)
 		)

Commit message: Fixed some R and C values, added missing 3D models
Parts:
- C20, C21: value 100uF -> 0.1uF
- C7: value 4.7uF -> 100uF
- R5: value R -> 10k
- moved C20 13.9 mm to (163.8, 54.8)
- moved C22 9.17 mm to (170.3, 55.2)
- moved C21 1.14 mm to (172.0, 46.1)
Other:
- board text added: "+"
Changed lines of the file:
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@@
 			)
 		)
+		(model "${KIPRJMOD}/libraries/NRF52832_QFAA_R/NRF52832-QFAA-R.step"
+			(offset
+				(xyz 0 0 0)
+			)
+			(scale
+				(xyz 1 1 1)
+			)
+			(rotate
+				(xyz -90 -0 -0)
+			)
+		)
 	)
 	(footprint "Capacitor_SMD:C_0603_1608Metric"
 		(layer "F.Cu")
-		(at 174.66 46.075 -90)
+		(at 163.77 54.765 -90)
 		(descr "Capacitor SMD 0603 (1608 Metric), square (rectangular) end terminal, IPC-7351 nominal, (Body size source: IPC-SM-782 page 76, https://www.pcb-3d.com/wordpress/wp-content/uploads/ipc-sm-782a_amendment_1_and_2.pdf), generated with kicad-footprint-generator")
 		(tags "capacitor")
 		(property "Reference" "C20"
-			(at -2.055 -1.69 180)
+			(at -0.435 2.24 180)
 			(layer "F.SilkS")
 			(effects
@@
 			)
 		)
-		(property "Value" "100uF"
+		(property "Value" "0.1uF"
 			(at 0 1.43 90)
 			(layer "F.Fab")
@@
 		(tags "capacitor")
 		(property "Reference" "C14"
-			(at 0.175 -1.35 0)
+			(at 2.825 -0.57 0)
 			(unlocked yes)
 			(layer "F.SilkS")
@@
 		(tags "capacitor")
 		(property "Reference" "C11"
-			(at 0.225 1.35 0)
+			(at 2.165 1.36 0)
 			(unlocked yes)
 			(layer "F.SilkS")
@@
 		)
 		(embedded_fonts no)
+		(model "${KIPRJMOD}/libraries/BME688/BME688.step"
+			(offset
+				(xyz 0 0 0)
+			)
+			(scale
+				(xyz 1 1 1)
+			)
+			(rotate
+				(xyz -90 -0 -180)
+			)
+		)
 	)
 	(footprint "Capacitor_SMD:C_0603_1608Metric"
@@
 			)
 		)
-		(property "Value" "R"
+		(property "Value" "10k"
 			(at 0 1.43 90)
 			(layer "F.Fab")
@@
 	(footprint "Capacitor_SMD:C_0603_1608Metric"
 		(layer "F.Cu")
-		(at 171.6 46.075 -90)
+		(at 170.33 55.155 -90)
 		(descr "Capacitor SMD 0603 (1608 Metric), square (rectangular) end terminal, IPC-7351 nominal, (Body size source: IPC-SM-782 page 76, https://www.pcb-3d.com/wordpress/wp-content/uploads/ipc-sm-782a_amendment_1_and_2.pdf), generated with kicad-footprint-generator")
 		(tags "capacitor")
 		(property "Reference" "C22"
-			(at 2.255 -0.49 0)
+			(at 1.725 -2.03 0)
 			(unlocked yes)
 			(layer "F.SilkS")
@@
 		(tags "capacitor")
 		(property "Reference" "C25"
-			(at 2.03 1.05 0)
+			(at 1.85 1.09 0)
 			(unlocked yes)
 			(layer "F.SilkS")
@@
 	(footprint "Capacitor_SMD:C_0603_1608Metric"
 		(layer "F.Cu")
-		(at 173.15 46.075 -90)
+		(at 172.01 46.115 -90)
 		(descr "Capacitor SMD 0603 (1608 Metric), square (rectangular) end terminal, IPC-7351 nominal, (Body size source: IPC-SM-782 page 76, https://www.pcb-3d.com/wordpress/wp-content/uploads/ipc-sm-782a_amendment_1_and_2.pdf), generated with kicad-footprint-generator")
 		(tags "capacitor")
@@
 			)
 		)
-		(property "Value" "100uF"
+		(property "Value" "0.1uF"
 			(at -2.445 1.45 90)
 			(layer "F.Fab")
@@
 		)
 		(embedded_fonts no)
+		(model "${KIPRJMOD}/libraries/SFV24R_2STE1HLF/SFV24R-2STE1HLF.step"
+			(offset
+				(xyz -8 -2 0)
+			)
+			(scale
+				(xyz 1 1 1)
+			)
+			(rotate
+				(xyz -90 -0 -0)
+			)
+		)
 	)
 	(footprint "Connector_JST:JST_PH_S2B-PH-SM4-TB_1x02-1MP_P2.00mm_Horizontal"
@@
 			)
 		)
+		(model "${KIPRJMOD}/libraries/S2B_PH_SM4_TB/S2B-PH-SM4-TB.step"
+			(offset
+				(xyz 0 -4.5 0)
+			)
+			(scale
+				(xyz 1 1 1)
+			)
+			(rotate
+				(xyz -90 -0 -0)
+			)
+		)
 	)
 	(footprint "Connector_USB:USB_C_Receptacle_GCT_USB4110"
@@
 			)
 		)
+		(model "${KIPRJMOD}/libraries/USB4110_GF_A/USB4110GFA.step"
+			(offset
+				(xyz 0 2.57 0)
+			)
+			(scale
+				(xyz 1 1 1)
+			)
+			(rotate
+				(xyz -90 -0 -0)
+			)
+		)
 	)
 	(footprint "Diode_SMD:D_SOD-523"
@@
 			)
 		)
-		(property "Value" "4.7uF"
+		(property "Value" "100uF"
 			(at 0 -1.43 90)
 			(layer "B.Fab")
@@
 		)
 	)
+	(gr_text "+"
+		(at 181.97 64.72 0)
+		(layer "B.SilkS")
+		(effects
+			(font
+				(size 1 1)
+				(thickness 0.1)
+			)
+			(justify left bottom)
+		)
+	)
 	(segment
 		(start 155.678274 53.59)
@@
 	)
 	(segment
+		(start 175.11 59.16)
+		(end 175.12 59.16)
+		(width 0.2)
+		(layer "F.Cu")
+		(net 3)
+	)
+	(segment
 		(start 168.16 41.15)
 		(end 170.2 41.15)
@@
 	)
 	(segment
-		(start 169.28 52.95)
-		(end 169.28 53.32)
+		(start 165.94 56.16)
+		(end 163.77 53.99)
 		(width 0.2)
 		(layer "F.Cu")
@@
 	)
 	(segment
-		(start 175.12 59.16)
-		(end 173.915 57.955)
+		(start 181.8875 72.89)
+		(end 180.75 72.89)
 		(width 0.2)
 		(layer "F.Cu")
@@
 	)
 	(segment
-		(start 173.915 57.955)
-		(end 170.04 54.08)
+		(start 169.28 52.95)
+		(end 169.28 53.33)
 		(width 0.2)
 		(layer "F.Cu")
@@
 	)
 	(segment
-		(start 181.8875 72.89)
-		(end 180.75 72.89)
+		(start 182.18 71.29)
+		(end 182.57 70.9)
 		(width 0.2)
 		(layer "F.Cu")
@@
 	)
 	(segment
-		(start 182.18 71.29)
-		(end 182.57 70.9)
+		(start 164.13 52.2)
+		(end 164.13 53.63)
+		(width 0.2)
+		(layer "F.Cu")
+		(net 3)
+	)
+	(segment
+		(start 164.13 53.63)
+		(end 163.77 53.99)
 		(width 0.2)
 		(layer "F.Cu")
@@
 	)
 	(segment
-		(start 171.46 62.82)
-		(end 169.42 62.82)
+		(start 169.28 53.33)
+		(end 170.33 54.38)
 		(width 0.2)
 		(layer "F.Cu")
@@
 	)
 	(segment
-		(start 164.13 52.2)
-		(end 164.13 54.44831)
+		(start 171.46 62.82)
+		(end 169.42 62.82)
 		(width 0.2)
 		(layer "F.Cu")
@@
 	)
 	(segment
+		(start 170.33 54.38)
+		(end 175.11 59.16)
+		(width 0.2)
+		(layer "F.Cu")
+		(net 3)
+	)
+	(segment
 		(start 176.59 45.3)
 		(end 179.49 45.3)
@@
 	)
 	(segment
-		(start 164.13 54.44831)
-		(end 165.94 56.25831)
+		(start 160.85 44.9)
+		(end 160.1747 45.5753)
 		(width 0.2)
 		(layer "F.Cu")
@@
 	)
 	(segment
-		(start 160.85 44.9)
-		(end 160.1747 45.5753)
+		(start 165.94 57.35)
+		(end 165.94 56.16)
 		(width 0.2)
 		(layer "F.Cu")
@@
 	)
 	(segment
-		(start 169.28 53.32)
-		(end 170.04 54.08)
-		(width 0.2)
-		(layer "F.Cu")
-		(net 3)
-	)
-	(segment
 		(start 165.94 57.35)
 		(end 165.94 63.86)
@@
 	)
 	(segment
-		(start 165.94 56.25831)
-		(end 165.94 57.35)
-		(width 0.2)
-		(layer "F.Cu")
-		(net 3)
-	)
-	(segment
 		(start 177.065 60.7825)
 		(end 177.065 62.195)
@@
 	)
 	(via
-		(at 170.04 54.08)
+		(at 170.33 54.38)
 		(size 0.6)
 		(drill 0.3)
@@
 	)
 	(segment
+		(start 170.33 54.38)
+		(end 168.91 54.38)
+		(width 0.2)
+		(layer "B.Cu")
+		(net 3)
+	)
+	(segment
 		(start 182 44.7)
 		(end 181.85 44.7)
@@
 	)
 	(segment
-		(start 165.94 57.35)
-		(end 169.21 54.08)
-		(width 0.2)
-		(layer "B.Cu")
-		(net 3)
-	)
-	(segment
 		(start 166.06 41.86)
 		(end 166.77 41.15)
@@
 	)
 	(segment
-		(start 169.21 54.08)
-		(end 170.04 54.08)
+		(start 168.91 54.38)
+		(end 165.94 57.35)
 		(width 0.2)
 		(layer "B.Cu")
@@
 	(segment
 		(start 172.4 55.1)
-		(end 170.03 52.73)
+		(end 172.4 54.84)
 		(width 0.2)
 		(layer "F.Cu")
@@
 	)
 	(segment
-		(start 170.03 52.73)
+		(start 170.03 52.47)
 		(end 170.03 52.2)
 		(width 0.2)
@@
 	)
 	(segment
+		(start 172.4 54.84)
+		(end 170.03 52.47)
+		(width 0.2)
+		(layer "F.Cu")
+		(net 8)
+	)
+	(segment
 		(start 160.9 54.7)
 		(end 160.9 56.2)
@@
 	)
 	(segment
-		(start 164.13 51.8)
+		(start 162.7 51.9513)
 		(end 162.8513 51.8)
 		(width 0.2)
@@
 	)
 	(segment
-		(start 162.8513 51.8)
-		(end 162.7 51.9513)
+		(start 164.25 58.995)
+		(end 164.215 59.03)
 		(width 0.2)
 		(layer "F.Cu")
@@
 	)
 	(segment
-		(start 164.25 55.45)
-		(end 162.7 53.9)
+		(start 164.04 57.5)
+		(end 162.7 56.16)
 		(width 0.2)
 		(layer "F.Cu")
@@
 	)
 	(segment
-		(start 164.25 58.995)
-		(end 164.215 59.03)
+		(start 162.8513 51.8)
+		(end 164.13 51.8)
 		(width 0.2)
 		(layer "F.Cu")
@@
 	(segment
 		(start 164.25 57.5)
-		(end 164.25 55.45)
+		(end 164.04 57.5)
 		(width 0.2)
 		(layer "F.Cu")
@@
 	)
 	(segment
-		(start 162.7 53.9)
+		(start 162.7 56.16)
 		(end 162.7 51.9513)
 		(width 0.2)
@@
 	)
 	(segment
+		(start 170.326 57.776322)
+		(end 170.326 57.806)
+		(width 0.2)
+		(layer "F.Cu")
+		(net 40)
+	)
+	(segment
+		(start 170.086178 57.5365)
+		(end 170.326 57.776322)
+		(width 0.2)
+		(layer "F.Cu")
+		(net 40)
+	)
+	(segment
 		(start 168.88 52.95)
-		(end 168.88 55.905)
+		(end 168.88 56.36)
+		(width 0.2)
+		(layer "F.Cu")
+		(net 40)
+	)
+	(segment
+		(start 170.0565 57.5365)
+		(end 170.086178 57.5365)
 		(width 0.2)
 		(layer "F.Cu")
@@
 	)
 	(segment
-		(start 168.88 55.905)
+		(start 168.88 56.36)
+		(end 170.0565 57.5365)
+		(width 0.2)
+		(layer "F.Cu")
+		(net 40)
+	)
+	(segment
+		(start 170.695 58.175)
 		(end 171.15 58.175)
 		(width 0.2)
 		(layer "F.Cu")
+		(net 40)
+	)
+	(segment
+		(start 170.326 57.806)
+		(end 170.695 58.175)
+		(width 0.2)
+		(layer "F.Cu")
