File: hardware/air-ctrl.kicad_pcb (KiCad board)
At the start: 2 copper layers, 35 x 35 mm, 71 parts, among them J1 USB_C_Receptacle_USB2.0_16P, J2 SFV24R-2STE1HLF, J3 Conn_ARM_SWD_TagConnect_TC203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, J4 Conn_01x02, Q1 BSS138, SW1 SW_RST, U1 nRF52832-QFxx, U2 BME688, U3 MCP73871-2CC, U4 MCP1700x-330xxTT, Y1 32MHz, Y2 32.768kHz

Commit message: Added ground pour on top and bottom layers, added via stitching
Parts:
- moved TP6 5.95 mm to (155.9, 68.5)
Routing:
- net -BATT: track 14.9 -> 22.3 mm, vias 0 -> 23
- net /power/V_BUS: track 22.8 -> 20.5 mm
- net /power/V_3V3: track 153.9 -> 152.7 mm
- added copper zone on B.Cu, net -BATT
- added copper zone on F.Cu, net -BATT
