File: hardware/power.kicad_sch (KiCad schematic)
At the start: 2 parts, among them U3 MCP73871-2CC, U4 MCP1700x-330xxTT

Commit message: fixed display schematic
Parts:
- added J1: USB_C_Receptacle_USB2.0_16P, symbol Connector:USB_C_Receptacle_USB2.0_16P
Connections:
- new net: J1.A4 (VBUS), J1.A9 (VBUS), J1.B4 (VBUS), J1.B9 (VBUS)
- new net: J1.A6 (D+), J1.B6 (D+)
- new net: J1.A7 (D-), J1.B7 (D-)
- new net GND: J1.A1 (GND), J1.A12 (GND), J1.B1 (GND), J1.B12 (GND), J1.S1 (SHIELD)
- no-connect marks 0 -> 4

Commit message: wip: power circuit
Parts:
- added C6, C7: 10uF, symbol Device:C
- added C8, C9: 1uF, symbol Device:C
- added F1: Polyfuse, symbol Device:Polyfuse
- added R10, R11, R12: 10k, symbol Device:R
- added R8, R9: 5.1k, symbol Device:R
Connections:
- net GND is gone; now on net -BATT: J1.A1 (GND), J1.A12 (GND), J1.B1 (GND), J1.B12 (GND), J1.S1 (SHIELD)
- net -BATT: now reaches U4.1 (GND)
- net -BATT: now also U3.10 (V_{SS}), U3.11 (V_{SS}), U3.21 (V_{SS}), U3.3 (SEL), U3.4 (PROG2), C6.2, C7.2, C8.2, C9.2, R10.2, R11.2, R12.2, R8.2, R9.2
- net V_3V3: now reaches U4.2 (VO)
- net V_3V3: now also C9.1
- net at U4.3 (VI): now also U3.1 (OUT), U3.20 (OUT), C8.1
- net V_BUS: now reaches J1.A4 (VBUS), J1.A9 (VBUS), J1.B4 (VBUS), J1.B9 (VBUS)
- net V_BUS: now also F1.1
- net at J1.A5 (CC1): now also R8.1
- net at J1.A6 (D+): no longer J1.B6 (D+)
- net at J1.A7 (D-): no longer J1.B7 (D-)
- net at J1.B5 (CC2): now also R9.1
- net at U3.12 (PROG3): now also R12.1
- net at U3.13 (PROG1): now also R10.1
- net +BATT: now reaches U3.14 (V_{BAT}), U3.15 (V_{BAT})
- net +BATT: now also U3.16 (V_{BAT_SENSE}), C7.1
- net V_IN: now reaches U3.17 (CE)
- net V_IN: now also U3.2 (VPCC), C6.1, F1.2
- net at U3.5 (THERM): now also U3.9 (~{TE}), R11.1
- no-connect marks 4 -> 6
Other:
- note added: "100mA charge current"
- moved on the sheet: J1, U3, U4

Commit message: finished first draft of schematic, need to review
Parts:
- added D1: CHG_LED, symbol Device:LED
- added D2: PWR_LED, symbol Device:LED
- added D3: LBAT_LED, symbol Device:LED
- added R13, R14, R15: 12k, symbol Device:R
Connections:
- net V_IN: now also U3.18 (IN), U3.19 (IN), D1.2 (A), D2.2 (A), D3.2 (A)
- net at U3.6 (~{PG}): now also R14.2
- net at U3.7 (STAT2): now also R13.2
- net at U3.8 (STAT1/~{LBO}): now also R15.2
- new net: D3.1 (K), R15.1
- new net: D2.1 (K), R14.1
- new net: D1.1 (K), R13.1
Other:
- note added: "Battery connector???"
- note added: "PG - Input power present STAT1 - Low battery indicator STAT2 - Charging indicator"
- moved on the sheet: C7, F1, J1, R8, R9

Commit message: fixed schematic
Parts:
- added J4: Conn_01x02, symbol Connector_Generic:Conn_01x02
- added TP1: TP_VBATT, symbol Connector:TestPoint
- added TP2: TP_VIN, symbol Connector:TestPoint
- added TP3: TP_VOUT, symbol Connector:TestPoint
- added TP4: TP_3V3, symbol Connector:TestPoint
- added TP5: TP_GND, symbol Connector:TestPoint
- added TP6: TP_VBUS, symbol Connector:TestPoint
- added U5: USBLC6-2SC6, Package_TO_SOT_SMD:SOT-23-6, symbol Power_Protection:USBLC6-2SC6
Connections:
- net +BATT: now also J4.1 (Pin_1), TP1.1
- net -BATT: now also J4.2 (Pin_2), TP5.1
- net V_3V3: now also TP4.1
- net V_BUS: now also TP6.1, U5.5 (VBUS); no longer F1.1
- net V_IN: now also TP2.1
- net at C8.1, U3.1 (OUT), U3.20 (OUT)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: now also TP3.1
- new net: F1.1, U5.2 (GND)
- no-connect marks 6 -> 10
Other:
- note added: "Battery connector"
- note added: "ESD protection"
- note removed: "Battery connector???"
- moved on the sheet: C7, D2, F1, R14

Commit message: changed to smd components, wip layout
Parts:
- C6, C7, C8, C9: footprint (none) -> Capacitor_SMD:C_0603_1608Metric
- D1, D2, D3: footprint (none) -> LED_SMD:LED_0805_2012Metric
- F1: footprint (none) -> Fuse:Fuse_1206_3216Metric
- J1: footprint (none) -> Connector_USB:USB_C_Receptacle_GCT_USB4110
- J4: footprint (none) -> Connector_JST:JST_PH_S2B-PH-SM4-TB_1x02-1MP_P2.00mm_Horizontal
- R10, R11, R12, R13, R14, R15, R8, R9: footprint (none) -> Resistor_SMD:R_0603_1608Metric
- TP1, TP2, TP3, TP4, TP5, TP6: footprint (none) -> TestPoint:TestPoint_Pad_D1.0mm
Changed lines of the file:
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@@
 			)
 		)
-		(property "Footprint" ""
+		(property "Footprint" "Capacitor_SMD:C_0603_1608Metric"
 			(at 220.6752 104.14 0)
 			(effects
@@
 			)
 		)
-		(property "Footprint" ""
+		(property "Footprint" "LED_SMD:LED_0805_2012Metric"
 			(at 194.31 118.11 0)
 			(effects
@@
 			)
 		)
-		(property "Footprint" ""
+		(property "Footprint" "TestPoint:TestPoint_Pad_D1.0mm"
 			(at 218.44 142.24 0)
 			(effects
@@
 			)
 		)
-		(property "Footprint" ""
+		(property "Footprint" "Resistor_SMD:R_0603_1608Metric"
 			(at 186.69 107.442 90)
 			(effects
@@
 			)
 		)
-		(property "Footprint" ""
+		(property "Footprint" "Capacitor_SMD:C_0603_1608Metric"
 			(at 223.2152 53.34 0)
 			(effects
@@
 			)
 		)
-		(property "Footprint" ""
+		(property "Footprint" "Resistor_SMD:R_0603_1608Metric"
 			(at 186.69 123.952 90)
 			(effects
@@
 			)
 		)
-		(property "Footprint" ""
+		(property "Footprint" "Connector_USB:USB_C_Receptacle_GCT_USB4110"
 			(at 71.12 57.15 0)
 			(effects
@@
 			)
 		)
-		(property "Footprint" ""
+		(property "Footprint" "Resistor_SMD:R_0603_1608Metric"
 			(at 134.62 106.172 90)
 			(effects
@@
 			)
 		)
-		(property "Footprint" ""
+		(property "Footprint" "Capacitor_SMD:C_0603_1608Metric"
 			(at 197.8152 53.34 0)
 			(effects
@@
 			)
 		)
-		(property "Footprint" ""
+		(property "Footprint" "Resistor_SMD:R_0603_1608Metric"
 			(at 99.822 52.07 90)
 			(effects
@@
 			)
 		)
-		(property "Footprint" ""
+		(property "Footprint" "TestPoint:TestPoint_Pad_D1.0mm"
 			(at 190.5 40.64 0)
 			(effects
@@
 			)
 		)
-		(property "Footprint" ""
+		(property "Footprint" "LED_SMD:LED_0805_2012Metric"
 			(at 194.31 109.22 0)
 			(effects
@@
 			)
 		)
-		(property "Footprint" ""
+		(property "Footprint" "Resistor_SMD:R_0603_1608Metric"
 			(at 186.69 116.332 90)
 			(effects
@@
 			)
 		)
-		(property "Footprint" ""
+		(property "Footprint" "Capacitor_SMD:C_0603_1608Metric"
 			(at 89.8652 100.33 0)
 			(effects
@@
 			)
 		)
-		(property "Footprint" ""
+		(property "Footprint" "TestPoint:TestPoint_Pad_D1.0mm"
 			(at 100.33 41.91 0)
 			(effects
@@
 			)
 		)
-		(property "Footprint" ""
+		(property "Footprint" "Connector_JST:JST_PH_S2B-PH-SM4-TB_1x02-1MP_P2.00mm_Horizontal"
 			(at 238.76 95.25 0)
 			(effects
@@
 			)
 		)
-		(property "Footprint" ""
+		(property "Footprint" "TestPoint:TestPoint_Pad_D1.0mm"
 			(at 228.6 45.72 0)
 			(effects
@@
 			)
 		)
-		(property "Footprint" ""
+		(property "Footprint" "TestPoint:TestPoint_Pad_D1.0mm"
 			(at 142.24 41.91 0)
 			(effects
@@
 			)
 		)
-		(property "Footprint" ""
+		(property "Footprint" "Resistor_SMD:R_0603_1608Metric"
 			(at 132.842 120.65 90)
 			(effects
@@
 			)
 		)
-		(property "Footprint" ""
+		(property "Footprint" "LED_SMD:LED_0805_2012Metric"
 			(at 194.31 125.73 0)
 			(effects
@@
 			)
 		)
-		(property "Footprint" ""
+		(property "Footprint" "Resistor_SMD:R_0603_1608Metric"
 			(at 90.932 53.34 90)
 			(effects
@@
 			)
 		)
-		(property "Footprint" ""
+		(property "Footprint" "TestPoint:TestPoint_Pad_D1.0mm"
 			(at 210.82 95.25 0)
 			(effects
@@
 			)
 		)
-		(property "Footprint" ""
+		(property "Footprint" "Fuse:Fuse_1206_3216Metric"
 			(at 139.7 40.64 0)
 			(effects
@@
 			)
 		)
-		(property "Footprint" ""
+		(property "Footprint" "Resistor_SMD:R_0603_1608Metric"
 			(at 108.712 107.95 90)
 			(effects

Commit message: change to 2-pin ESD protection diode
Parts:
- removed U5: USBLC6-2SC6, Package_TO_SOT_SMD:SOT-23-6, symbol Power_Protection:USBLC6-2SC6
- added C24: 100nF, Capacitor_SMD:C_0603_1608Metric, symbol Device:C
- added D4: ESD5Zxx, Diode_SMD:D_SOD-523, symbol Diode:ESD5Zxx
Connections:
- net -BATT: now also C24.2, D4.2 (A)
- net V_BUS: now also F1.1, C24.1, D4.1 (K)
- no-connect marks 10 -> 6

Commit message: Fixed layout bottom layer
Also fixed all DRC issues
Parts:
- C7: value 10uF -> 4.7uF
Changed lines of the file:
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@@
 			)
 		)
-		(property "Value" "10uF"
+		(property "Value" "4.7uF"
 			(at 223.52 101.5999 0)
 			(effects

Commit message: routing power lines, fixing schematic
using 3.3V to power LEDs, fixed  CE-pin to be low
Connections:
- net -BATT: now also U3.9 (~{TE})
- net V_3V3: now also D1.2 (A), D2.2 (A), D3.2 (A)
- net V_IN: no longer D1.2 (A), D2.2 (A), D3.2 (A)
- net at R11.1, U3.5 (THERM): no longer U3.9 (~{TE})
Other:
- moved on the sheet: R11
Changed lines of the file:
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@@
 	)
 	(junction
-		(at 147.32 113.03)
-		(diameter 0)
-		(color 0 0 0 0)
-	)
-	(junction
 		(at 196.85 45.72)
 		(diameter 0)
@@
 	(wire
 		(pts
-			(xy 134.62 113.03) (xy 134.62 116.84)
+			(xy 128.27 113.03) (xy 128.27 116.84)
 		)
 		(stroke
@@
 	(wire
 		(pts
-			(xy 226.06 142.24) (xy 213.36 142.24)
+			(xy 140.97 118.11) (xy 140.97 121.92)
 		)
 		(stroke
@@
 	(wire
 		(pts
-			(xy 59.69 80.01) (xy 63.5 80.01)
+			(xy 226.06 142.24) (xy 213.36 142.24)
 		)
 		(stroke
@@
 	(wire
 		(pts
-			(xy 226.06 107.95) (xy 226.06 142.24)
+			(xy 59.69 80.01) (xy 63.5 80.01)
 		)
 		(stroke
@@
 	(wire
 		(pts
-			(xy 160.02 142.24) (xy 165.1 142.24)
+			(xy 226.06 107.95) (xy 226.06 142.24)
 		)
 		(stroke
@@
 	(wire
 		(pts
-			(xy 182.88 120.65) (xy 182.88 125.73)
+			(xy 160.02 142.24) (xy 165.1 142.24)
 		)
 		(stroke
@@
 	(wire
 		(pts
-			(xy 147.32 113.03) (xy 147.32 118.11)
+			(xy 182.88 120.65) (xy 182.88 125.73)
 		)
 		(stroke
@@
 	(wire
 		(pts
-			(xy 134.62 113.03) (xy 147.32 113.03)
+			(xy 128.27 113.03) (xy 147.32 113.03)
 		)
 		(stroke
@@
 	(wire
 		(pts
+			(xy 147.32 118.11) (xy 140.97 118.11)
+		)
+		(stroke
+			(width 0)
+			(type default)
+		)
+	)
+	(wire
+		(pts
 			(xy 196.85 45.72) (xy 203.2 45.72)
 		)
@@
 		)
 	)
-	(label "V_IN"
+	(label "V_3V3"
 		(at 212.09 118.11 0)
 		(effects
@@
 	)
 	(symbol
+		(lib_id "power:GND")
+		(at 140.97 121.92 0)
+		(unit 1)
+		(exclude_from_sim no)
+		(in_bom yes)
+		(on_board yes)
+		(dnp no)
+		(fields_autoplaced yes)
+		(property "Reference" "#PWR035"
+			(at 140.97 128.27 0)
+			(effects
+				(font
+					(size 1.27 1.27)
+				)
+				(hide yes)
+			)
+		)
+		(property "Value" "GND"
+			(at 140.97 127 0)
+			(effects
+				(font
+					(size 1.27 1.27)
+				)
+			)
+		)
+		(property "Footprint" ""
+			(at 140.97 121.92 0)
+			(effects
+				(font
+					(size 1.27 1.27)
+				)
+				(hide yes)
+			)
+		)
+		(property "Datasheet" ""
+			(at 140.97 121.92 0)
+			(effects
+				(font
+					(size 1.27 1.27)
+				)
+				(hide yes)
+			)
+		)
+		(property "Description" "Power symbol creates a global label with name \"GND\" , ground"
+			(at 140.97 121.92 0)
+			(effects
+				(font
+					(size 1.27 1.27)
+				)
+				(hide yes)
+			)
+		)
+		(pin "1"
+		)
+		(instances
+			(project "air-ctrl"
+				(path "/0ac49f41-390f-45da-b336-186a486bd4d5/4fb608f5-b95a-4746-b766-66c68a4f5c7d"
+					(reference "#PWR035")
+					(unit 1)
+				)
+			)
+		)
+	)
+	(symbol
 		(lib_id "Device:R")
 		(at 186.69 118.11 270)
@@
 	(symbol
 		(lib_id "power:GND")
-		(at 134.62 124.46 0)
+		(at 128.27 124.46 0)
 		(unit 1)
 		(exclude_from_sim no)
@@
 		(fields_autoplaced yes)
 		(property "Reference" "#PWR020"
-			(at 134.62 130.81 0)
+			(at 128.27 130.81 0)
 			(effects
 				(font
@@
 		)
 		(property "Value" "GND"
-			(at 134.62 129.54 0)
+			(at 128.27 129.54 0)
 			(effects
 				(font
@@
 		)
 		(property "Footprint" ""
-			(at 134.62 124.46 0)
+			(at 128.27 124.46 0)
 			(effects
 				(font
@@
 		)
 		(property "Datasheet" ""
-			(at 134.62 124.46 0)
+			(at 128.27 124.46 0)
 			(effects
 				(font
@@
 		)
 		(property "Description" "Power symbol creates a global label with name \"GND\" , ground"
-			(at 134.62 124.46 0)
+			(at 128.27 124.46 0)
 			(effects
 				(font
@@
 	(symbol
 		(lib_id "Device:R")
-		(at 134.62 120.65 0)
+		(at 128.27 120.65 0)
 		(unit 1)
 		(exclude_from_sim no)
@@
 		(fields_autoplaced yes)
 		(property "Reference" "R11"
-			(at 137.16 119.3799 0)
+			(at 130.81 119.3799 0)
 			(effects
 				(font
@@
 		)
 		(property "Value" "10k"
-			(at 137.16 121.9199 0)
+			(at 130.81 121.9199 0)
 			(effects
 				(font
@@
 		)
 		(property "Footprint" "Resistor_SMD:R_0603_1608Metric"
-			(at 132.842 120.65 90)
+			(at 126.492 120.65 90)
 			(effects
 				(font
@@
 		)
 		(property "Datasheet" "~"
-			(at 134.62 120.65 0)
+			(at 128.27 120.65 0)
 			(effects
 				(font
@@
 		)
 		(property "Description" "Resistor"
-			(at 134.62 120.65 0)
+			(at 128.27 120.65 0)
 			(effects
 				(font
