File: hardware/air-ctrl.kicad_sch (KiCad schematic)
At the start: 0 parts

Commit message: wip schematic
hierarchy and importing components
Other:
- added sheet connectors (connectors.kicad_sch)
- added sheet display (display.kicad_sch)
- added sheet mcu (mcu.kicad_sch)
- added sheet power (power.kicad_sch)
- added sheet sensor (sensor.kicad_sch)
Changed lines of the file:
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@@
 	(generator_version "9.0")
 	(paper "A4")
+	(sheet
+		(at 119.38 46.99)
+		(size 40.64 58.42)
+		(exclude_from_sim no)
+		(in_bom yes)
+		(on_board yes)
+		(dnp no)
+		(fields_autoplaced yes)
+		(stroke
+			(width 0.1524)
+			(type solid)
+		)
+		(fill
+			(color 0 0 0 0.0000)
+		)
+		(property "Sheetname" "mcu"
+			(at 119.38 46.2784 0)
+			(effects
+				(font
+					(size 1.27 1.27)
+				)
+				(justify left bottom)
+			)
+		)
+		(property "Sheetfile" "mcu.kicad_sch"
+			(at 119.38 105.9946 0)
+			(effects
+				(font
+					(size 1.27 1.27)
+				)
+				(justify left top)
+			)
+		)
+		(instances
+			(project "air-ctrl"
+				(path "/0ac49f41-390f-45da-b336-186a486bd4d5"
+					(page "2")
+				)
+			)
+		)
+	)
+	(sheet
+		(at 194.31 57.15)
+		(size 27.94 54.61)
+		(exclude_from_sim no)
+		(in_bom yes)
+		(on_board yes)
+		(dnp no)
+		(fields_autoplaced yes)
+		(stroke
+			(width 0.1524)
+			(type solid)
+		)
+		(fill
+			(color 0 0 0 0.0000)
+		)
+		(property "Sheetname" "power"
+			(at 194.31 56.4384 0)
+			(effects
+				(font
+					(size 1.27 1.27)
+				)
+				(justify left bottom)
+			)
+		)
+		(property "Sheetfile" "power.kicad_sch"
+			(at 194.31 112.3446 0)
+			(effects
+				(font
+					(size 1.27 1.27)
+				)
+				(justify left top)
+			)
+		)
+		(instances
+			(project "air-ctrl"
+				(path "/0ac49f41-390f-45da-b336-186a486bd4d5"
+					(page "3")
+				)
+			)
+		)
+	)
+	(sheet
+		(at 35.56 114.3)
+		(size 40.64 34.29)
+		(exclude_from_sim no)
+		(in_bom yes)
+		(on_board yes)
+		(dnp no)
+		(fields_autoplaced yes)
+		(stroke
+			(width 0.1524)
+			(type solid)
+		)
+		(fill
+			(color 0 0 0 0.0000)
+		)
+		(property "Sheetname" "display"
+			(at 35.56 113.5884 0)
+			(effects
+				(font
+					(size 1.27 1.27)
+				)
+				(justify left bottom)
+			)
+		)
+		(property "Sheetfile" "display.kicad_sch"
+			(at 35.56 149.1746 0)
+			(effects
+				(font
+					(size 1.27 1.27)
+				)
+				(justify left top)
+			)
+		)
+		(instances
+			(project "air-ctrl"
+				(path "/0ac49f41-390f-45da-b336-186a486bd4d5"
+					(page "6")
+				)
+			)
+		)
+	)
+	(sheet
+		(at 237.49 57.15)
+		(size 20.32 53.34)
+		(exclude_from_sim no)
+		(in_bom yes)
+		(on_board yes)
+		(dnp no)
+		(fields_autoplaced yes)
+		(stroke
+			(width 0.1524)
+			(type solid)
+		)
+		(fill
+			(color 0 0 0 0.0000)
+		)
+		(property "Sheetname" "connectors"
+			(at 237.49 56.4384 0)
+			(effects
+				(font
+					(size 1.27 1.27)
+				)
+				(justify left bottom)
+			)
+		)
+		(property "Sheetfile" "connectors.kicad_sch"
+			(at 237.49 111.0746 0)
+			(effects
+				(font
+					(size 1.27 1.27)
+				)
+				(justify left top)
+			)
+		)
+		(instances
+			(project "air-ctrl"
+				(path "/0ac49f41-390f-45da-b336-186a486bd4d5"
+					(page "4")
+				)
+			)
+		)
+	)
+	(sheet
+		(at 36.83 52.07)
+		(size 38.1 34.29)
+		(exclude_from_sim no)
+		(in_bom yes)
+		(on_board yes)
+		(dnp no)
+		(fields_autoplaced yes)
+		(stroke
+			(width 0.1524)
+			(type solid)
+		)
+		(fill
+			(color 0 0 0 0.0000)
+		)
+		(property "Sheetname" "sensor"
+			(at 36.83 51.3584 0)
+			(effects
+				(font
+					(size 1.27 1.27)
+				)
+				(justify left bottom)
+			)
+		)
+		(property "Sheetfile" "sensor.kicad_sch"
+			(at 36.83 86.9446 0)
+			(effects
+				(font
+					(size 1.27 1.27)
+				)
+				(justify left top)
+			)
+		)
+		(instances
+			(project "air-ctrl"
+				(path "/0ac49f41-390f-45da-b336-186a486bd4d5"
+					(page "5")
+				)
+			)
+		)
+	)
 	(sheet_instances
 		(path "/"

Commit message: fixed display schematic
Other:
- removed sheet connectors
- sheet display ports: added 3V3, DISP_BL, DISP_CS, DISP_MOSI, DISP_RST, DISP_SCLK; removed none
Changed lines of the file:
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@@
 	(paper "A4")
 	(sheet
-		(at 119.38 46.99)
+		(at 121.92 53.34)
 		(size 40.64 58.42)
 		(exclude_from_sim no)
@@
 		)
 		(property "Sheetname" "mcu"
-			(at 119.38 46.2784 0)
+			(at 121.92 52.6284 0)
 			(effects
 				(font
@@
 		)
 		(property "Sheetfile" "mcu.kicad_sch"
-			(at 119.38 105.9946 0)
+			(at 121.92 112.3446 0)
 			(effects
 				(font
@@
 	)
 	(sheet
-		(at 194.31 57.15)
+		(at 208.28 58.42)
 		(size 27.94 54.61)
 		(exclude_from_sim no)
@@
 		)
 		(property "Sheetname" "power"
-			(at 194.31 56.4384 0)
+			(at 208.28 57.7084 0)
 			(effects
 				(font
@@
 		)
 		(property "Sheetfile" "power.kicad_sch"
-			(at 194.31 112.3446 0)
+			(at 208.28 113.6146 0)
 			(effects
 				(font
@@
 			)
 		)
+		(pin "3V3" input
+			(at 76.2 118.11 0)
+			(effects
+				(font
+					(size 1.27 1.27)
+				)
+				(justify right)
+			)
+		)
+		(pin "DISP_CS" input
+			(at 76.2 123.19 0)
+			(effects
+				(font
+					(size 1.27 1.27)
+				)
+				(justify right)
+			)
+		)
+		(pin "DISP_BL" input
+			(at 76.2 127 0)
+			(effects
+				(font
+					(size 1.27 1.27)
+				)
+				(justify right)
+			)
+		)
+		(pin "DISP_RST" input
+			(at 76.2 130.81 0)
+			(effects
+				(font
+					(size 1.27 1.27)
+				)
+				(justify right)
+			)
+		)
+		(pin "DISP_SCLK" input
+			(at 76.2 134.62 0)
+			(effects
+				(font
+					(size 1.27 1.27)
+				)
+				(justify right)
+			)
+		)
+		(pin "DISP_MOSI" input
+			(at 76.2 138.43 0)
+			(effects
+				(font
+					(size 1.27 1.27)
+				)
+				(justify right)
+			)
+		)
 		(instances
 			(project "air-ctrl"
@@
 				)
 			)
-		)
-	)
-	(sheet
-		(at 237.49 57.15)
-		(size 20.32 53.34)
-		(exclude_from_sim no)
-		(in_bom yes)
-		(on_board yes)
-		(dnp no)
-		(fields_autoplaced yes)
-		(stroke
-			(width 0.1524)
-			(type solid)
-		)
-		(fill
-			(color 0 0 0 0.0000)
-		)
-		(property "Sheetname" "connectors"
-			(at 237.49 56.4384 0)
-			(effects
-				(font
-					(size 1.27 1.27)
-				)
-				(justify left bottom)
-			)
-		)
-		(property "Sheetfile" "connectors.kicad_sch"
-			(at 237.49 111.0746 0)
-			(effects
-				(font
-					(size 1.27 1.27)
-				)
-				(justify left top)
-			)
-		)
-		(instances
-			(project "air-ctrl"
-				(path "/0ac49f41-390f-45da-b336-186a486bd4d5"
-					(page "4")
-				)
-			)

Commit message: implemented sensor circuit
Other:
- sheet sensor ports: added I2C_SCL, I2C_SDA, VDD_3V3; removed none
Changed lines of the file:
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@@
+			)
+		)
+		(pin "VDD_3V3" input
+			(at 74.93 57.15 0)
+			(effects
+				(font
+					(size 1.27 1.27)
+				)
+				(justify right)
+			)
+		)
+		(pin "I2C_SDA" input
+			(at 74.93 67.31 0)
+			(effects
+				(font
+					(size 1.27 1.27)
+				)
+				(justify right)
+			)
+		)
+		(pin "I2C_SCL" input
+			(at 74.93 72.39 0)
+			(effects
+				(font
+					(size 1.27 1.27)
+				)
+				(justify right)
 			)
 		)

Commit message: finished first draft of schematic, need to review
Other:
- sheet display ports: added DISP_DC; removed none
- sheet mcu ports: added 3V3, DISP_BL, DISP_CS, DISP_DC, DISP_MOSI, DISP_RST, DISP_SCLK, I2C_SCL, I2C_SDA; removed none
- sheet power ports: added V_3V3; removed none

Commit message: Added name and revision
Other:
- title: (none) -> air-ctrl
Changed lines of the file:
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@@
 	(generator_version "9.0")
 	(paper "A4")
+	(title_block
+		(title "air-ctrl")
+		(date "2025-10-18")
+		(rev "1.1")
+	)
 	(junction
 		(at 176.53 62.23)
