File: hardware/sensor.kicad_sch (KiCad schematic)
At the start: 1 part, among them U2 BME688

Commit message: implemented sensor circuit
Parts:
- added C4: 0.1uF, symbol Device:C
- added C5: 4.7uF, symbol Device:C
- added R6, R7: 4.7k, symbol Device:R
Connections:
- net GND: now reaches U2.1 (GND)
- net GND: now also U2.5 (SDO), U2.7 (GND__1), C4.2, C5.2
- net VDD_3V3: now reaches U2.2 (CSB)
- net VDD_3V3: now also U2.6 (VDDIO), U2.8 (VDD), C4.1, C5.1, R6.1, R7.1
- net I2C_SDA: now reaches U2.3 (SDI)
- net I2C_SDA: now also R6.2
- net I2C_SCL: now reaches U2.4 (SCK)
- net I2C_SCL: now also R7.2

Commit message: changed to smd components, wip layout
Parts:
- C4, C5: footprint (none) -> Capacitor_SMD:C_0603_1608Metric
- R6, R7: footprint (none) -> Resistor_SMD:R_0603_1608Metric
Changed lines of the file:
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@@
 			)
 		)
-		(property "Footprint" ""
+		(property "Footprint" "Capacitor_SMD:C_0603_1608Metric"
 			(at 182.5752 68.58 0)
 			(effects
@@
 			)
 		)
-		(property "Footprint" ""
+		(property "Footprint" "Capacitor_SMD:C_0603_1608Metric"
 			(at 169.8752 68.58 0)
 			(effects
@@
 			)
 		)
-		(property "Footprint" ""
+		(property "Footprint" "Resistor_SMD:R_0603_1608Metric"
 			(at 195.072 73.66 90)
 			(effects
@@
 			)
 		)
-		(property "Footprint" ""
+		(property "Footprint" "Resistor_SMD:R_0603_1608Metric"
 			(at 118.872 78.74 90)
 			(effects

Commit message: Added name and revision
Other:
- title: (none) -> air-ctrl
Changed lines of the file:
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@@
 	(generator_version "9.0")
 	(paper "A4")
+	(title_block
+		(title "air-ctrl")
+		(date "2025-10-18")
+		(rev "1.1")
+	)
 	(junction
 		(at 196.85 83.82)
