File: hardware/display.kicad_sch (KiCad schematic)
At the start: 0 parts

Commit message: fixed display schematic
Parts:
- added C1, C2: 10uF, symbol Device:C
- added C3: 0.1uF, symbol Device:C
- added J2: SFV24R-2STE1HLF, SFV24R-2STE1HLF:AMPHENOL_SFV24R-2STE1HLF, symbol SFV24R-2STE1HLF:SFV24R-2STE1HLF
- added Q1: BSS138, Package_TO_SOT_SMD:SOT-23, symbol Transistor_FET:BSS138
- added R1, R2: 10k, symbol Device:R
- added R3, R4: 33, symbol Device:R
- added R5: R, symbol Device:R
Connections:
- new net: J2.12 (SDA), R3.2
- new net: J2.9 (DC), R4.2
- new net 3V3: C1.1, C2.1, C3.1, J2.1 (LEDA), J2.10 (WR), J2.4 (VDD2.8V), J2.5 (IOVCC1.8V), J2.6 (IM1/2), R1.1, R2.1, R5.1
- new net DISP_BL: Q1.1 (G), R5.2
- new net DISP_CS: J2.8 (CS), R2.2
- new net DISP_MOSI: R3.1
- new net DISP_RST: J2.7 (RESET), R1.2
- new net DISP_SCLK: R4.1
- new net GND: C1.2, C2.2, C3.2, J2.11 (RD), J2.13 (DB0), J2.14 (DB1), J2.15 (DB2), J2.16 (DB3), J2.17 (DB4), J2.18 (DB5), J2.19 (DB6), J2.20 (DB7), J2.23 (GND), J2.24 (GND), J2.3 (GND), J2.S1 (SHIELD), J2.S2 (SHIELD__1), Q1.2 (S)
- new net LEDK: J2.2 (LEDK), Q1.3 (D)
- no-connect marks 0 -> 2
Other:
- note added: "Switch to PWM the backlight"
- note added: "To select 4-SPI (1 bit) - pull high"
- note added: "decoupling capacitors to protect the IC from voltage fluctuations and noise on power line"
- note added: "to disable display during MCU reset"

Commit message: finished first draft of schematic, need to review
Connections:
- net 3V3: no longer J2.10 (WR)
- new net DISP_DC: J2.10 (WR)
Other:
- moved on the sheet: C1, C2, C3, Q1, R5

Commit message: changed to smd components, wip layout
Parts:
- removed R3, R4: 33, symbol Device:R
- C1, C2, C3: footprint (none) -> Capacitor_SMD:C_0603_1608Metric
- J2: footprint SFV24R-2STE1HLF:AMPHENOL_SFV24R-2STE1HLF -> SFV24R_2STE1HLF:AMPHENOL_SFV24R-2STE1HLF
- R1, R2, R5: footprint (none) -> Resistor_SMD:R_0603_1608Metric
Connections:
- net DISP_MOSI: now also J2.12 (SDA)
- net DISP_SCLK: now also J2.9 (DC)
Changed lines of the file:
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@@
 	(wire
 		(pts
-			(xy 163.83 71.12) (xy 160.02 71.12)
+			(xy 161.29 67.31) (xy 189.23 67.31)
 		)
 		(stroke
@@
 	(wire
 		(pts
-			(xy 172.72 59.69) (xy 189.23 59.69)
-		)
-		(stroke
-			(width 0)
-			(type default)
-		)
-	)
-	(wire
-		(pts
 			(xy 77.47 104.14) (xy 77.47 109.22)
 		)
@@
 	(wire
 		(pts
-			(xy 172.72 67.31) (xy 189.23 67.31)
-		)
-		(stroke
-			(width 0)
-			(type default)
-		)
-	)
-	(wire
-		(pts
-			(xy 172.72 71.12) (xy 172.72 67.31)
-		)
-		(stroke
-			(width 0)
-			(type default)
-		)
-	)
-	(wire
-		(pts
 			(xy 177.8 105.41) (xy 189.23 105.41)
 		)
@@
 	(wire
 		(pts
-			(xy 161.29 59.69) (xy 165.1 59.69)
+			(xy 161.29 59.69) (xy 189.23 59.69)
 		)
 		(stroke
@@
 	(wire
 		(pts
-			(xy 172.72 71.12) (xy 171.45 71.12)
-		)
-		(stroke
-			(width 0)
-			(type default)
-		)
-	)
-	(wire
-		(pts
-			(xy 176.53 63.5) (xy 176.53 62.23)
-		)
-		(stroke
-			(width 0)
-			(type default)
-		)
-	)
-	(wire
-		(pts
 			(xy 175.26 52.07) (xy 175.26 49.53)
 		)
@@
 	(wire
 		(pts
-			(xy 161.29 63.5) (xy 176.53 63.5)
+			(xy 161.29 62.23) (xy 189.23 62.23)
 		)
 		(stroke
@@
 		(pts
 			(xy 189.23 46.99) (xy 175.26 46.99)
-		)
-		(stroke
-			(width 0)
-			(type default)
-		)
-	)
-	(wire
-		(pts
-			(xy 176.53 62.23) (xy 189.23 62.23)
 		)
 		(stroke
@@
 	(hierarchical_label "DISP_MOSI"
 		(shape input)
-		(at 160.02 71.12 180)
+		(at 161.29 67.31 180)
 		(effects
 			(font
@@
 	(hierarchical_label "DISP_DC"
 		(shape input)
-		(at 161.29 63.5 180)
+		(at 161.29 62.23 180)
 		(effects
 			(font
@@
 			)
 			(justify right)
-		)
-	)
-	(symbol
-		(lib_id "Device:R")
-		(at 167.64 71.12 90)
-		(unit 1)
-		(exclude_from_sim no)
-		(in_bom yes)
-		(on_board yes)
-		(dnp no)
-		(property "Reference" "R3"
-			(at 167.64 66.04 90)
-			(effects
-				(font
-					(size 1.27 1.27)
-				)
-			)
-		)
-		(property "Value" "33"
-			(at 167.64 68.834 90)
-			(effects
-				(font
-					(size 1.27 1.27)
-				)
-			)
-		)
-		(property "Footprint" ""
-			(at 167.64 72.898 90)
-			(effects
-				(font
-					(size 1.27 1.27)
-				)
-				(hide yes)
-			)
-		)
-		(property "Datasheet" "~"
-			(at 167.64 71.12 0)
-			(effects
-				(font
-					(size 1.27 1.27)
-				)
-				(hide yes)
-			)
-		)
-		(property "Description" "Resistor"
-			(at 167.64 71.12 0)
-			(effects
-				(font
-					(size 1.27 1.27)
-				)
-				(hide yes)
-			)
-		)
-		(pin "1"
-		)
-		(pin "2"
-		)
-		(instances
-			(project ""
-				(path "/0ac49f41-390f-45da-b336-186a486bd4d5/54858e69-cc47-4c61-af10-9f8f625aa872"
-					(reference "R3")
-					(unit 1)
-				)
-			)
-		)
-	)
-	(symbol
-		(lib_id "Device:R")
-		(at 168.91 59.69 90)
-		(unit 1)
-		(exclude_from_sim no)
-		(in_bom yes)
-		(on_board yes)
-		(dnp no)
-		(fields_autoplaced yes)
-		(property "Reference" "R4"
-			(at 168.91 53.34 90)
-			(effects
-				(font
-					(size 1.27 1.27)
-				)
-			)
-		)
-		(property "Value" "33"
-			(at 168.91 55.88 90)
-			(effects
-				(font
-					(size 1.27 1.27)
-				)
-			)
-		)
-		(property "Footprint" ""
-			(at 168.91 61.468 90)
-			(effects
-				(font
-					(size 1.27 1.27)
-				)
-				(hide yes)
-			)
-		)
-		(property "Datasheet" "~"
-			(at 168.91 59.69 0)
-			(effects
-				(font
-					(size 1.27 1.27)
-				)
-				(hide yes)
-			)
-		)
-		(property "Description" "Resistor"
-			(at 168.91 59.69 0)
-			(effects
-				(font
-					(size 1.27 1.27)
-				)
-				(hide yes)
-			)
-		)
-		(pin "1"
-		)
-		(pin "2"
-		)
-		(instances
-			(project ""
-				(path "/0ac49f41-390f-45da-b336-186a486bd4d5/54858e69-cc47-4c61-af10-9f8f625aa872"
-					(reference "R4")
-					(unit 1)
-				)
-			)
 		)
 	)
@@
 			)
 		)
-		(property "Footprint" ""
+		(property "Footprint" "Resistor_SMD:R_0603_1608Metric"
 			(at 150.622 46.99 90)
 			(effects
@@
 			)
 		)
-		(property "Footprint" ""
+		(property "Footprint" "Resistor_SMD:R_0603_1608Metric"
 			(at 140.462 46.99 90)
 			(effects
@@
 			)
 		)
-		(property "Footprint" ""
+		(property "Footprint" "Capacitor_SMD:C_0603_1608Metric"
 			(at 96.2152 48.26 0)
 			(effects
@@
 			)
 		)
-		(property "Footprint" "SFV24R-2STE1HLF:AMPHENOL_SFV24R-2STE1HLF"
+		(property "Footprint" "SFV24R_2STE1HLF:AMPHENOL_SFV24R-2STE1HLF"
 			(at 199.39 72.39 0)
 			(effects
@@
 			)
 		)
-		(property "Footprint" ""
+		(property "Footprint" "Resistor_SMD:R_0603_1608Metric"
 			(at 60.452 91.44 90)
 			(effects
@@
 			)
 		)
-		(property "Footprint" ""
+		(property "Footprint" "Capacitor_SMD:C_0603_1608Metric"
 			(at 73.3552 48.26 0)
 			(effects
@@
 			)
 		)
-		(property "Footprint" ""
+		(property "Footprint" "Capacitor_SMD:C_0603_1608Metric"
 			(at 84.7852 48.26 0)
 			(effects

Commit message: Added name and revision
Other:
- title: (none) -> air-ctrl
Changed lines of the file:
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@@
 	(generator_version "9.0")
 	(paper "A4")
+	(title_block
+		(title "air-ctrl")
+		(date "2025-10-18")
+		(rev "1.1")
+	)
 	(text "to disable display during MCU reset"
 		(exclude_from_sim no)

Commit message: Fixed some R and C values, added missing 3D models
Parts:
- R5: value R -> 10k
Changed lines of the file:
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@@
 			)
 		)
-		(property "Value" "R"
+		(property "Value" "10k"
 			(at 64.77 92.7099 0)
 			(effects
