File: hardware/mcu.kicad_sch (KiCad schematic)
At the start: 1 part, among them U1 nRF52832-QFxx

Commit message: fixed display schematic
Parts:
- added J3: Conn_ARM_SWD_TagConnect_TC2030-NL, Connector:Tag-Connect_TC2030-IDC-NL_2x03_P1.27mm_Vertical, symbol Connector:Conn_ARM_SWD_TagConnect_TC2030-NL
Changed lines of the file:
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@@
-		)
-	)
-	(hierarchical_label "GND"
-		(shape input)
-		(at 219.71 64.77 0)
-		(effects
-			(font
-				(size 1.27 1.27)
-			)
-			(justify left)
 		)
 	)
@@
 					(unit 1)
 				)
+			)
+		)
+	)
+	(symbol
+		(lib_id "Connector:Conn_ARM_SWD_TagConnect_TC2030-NL")
+		(at 62.23 114.3 0)
+		(unit 1)
+		(exclude_from_sim no)
+		(in_bom no)
+		(on_board yes)
+		(dnp no)
+		(fields_autoplaced yes)
+		(property "Reference" "J3"
+			(at 55.88 113.0299 0)
+			(effects
+				(font
+					(size 1.27 1.27)
+				)
+				(justify right)
+			)
+		)
+		(property "Value" "Conn_ARM_SWD_TagConnect_TC2030-NL"
+			(at 55.88 115.5699 0)
+			(effects
+				(font
+					(size 1.27 1.27)
+				)
+				(justify right)
+			)
+		)
+		(property "Footprint" "Connector:Tag-Connect_TC2030-IDC-NL_2x03_P1.27mm_Vertical"
+			(at 62.23 132.08 0)
+			(effects
+				(font
+					(size 1.27 1.27)
+				)
+				(hide yes)
+			)
+		)
+		(property "Datasheet" "https://www.tag-connect.com/wp-content/uploads/bsk-pdf-manager/TC2030-CTX_1.pdf"
+			(at 62.23 129.54 0)
+			(effects
+				(font
+					(size 1.27 1.27)
+				)
+				(hide yes)
+			)
+		)
+		(property "Description" "Tag-Connect ARM Cortex SWD JTAG connector, 6 pin, no legs"
+			(at 62.23 114.3 0)
+			(effects
+				(font
+					(size 1.27 1.27)
+				)
+				(hide yes)
+			)
+		)
+		(pin "1"
+		)
+		(pin "2"
+		)
+		(pin "6"
+		)
+		(pin "5"
+		)
+		(pin "3"
+		)
+		(pin "4"
+		)
+		(instances
+			(project "air-ctrl"
+				(path "/0ac49f41-390f-45da-b336-186a486bd4d5/1bbfc266-7a13-4dd4-be44-db318575809d"
+					(reference "J3")
+					(unit 1)
+				)

Commit message: finished first draft of schematic, need to review
Parts:
- added AE1: BLE, symbol Device:Antenna_Shield
- added C10, C11: 100nF, symbol Device:C
- added C12: 100pF, symbol Device:C
- added C13, C14, C15, C16: 12pF, symbol Device:C
- added C17, C19: 0.8pF, symbol Device:C_Small
- added C18: 1uF, symbol Device:C
- added C20, C21: 100uF, symbol Device:C_Small
- added C22: 4.7uF, symbol Device:C_Small
- added L1: 3.9nH, symbol Device:L_Small
- added L2: 10uH, symbol Device:L_Small
- added L3: 15uH, symbol Device:L_Small
- added R16: 0R, symbol Device:R_Small
- added Y1: 32MHz, symbol Device:Crystal_GND24
- added Y2: 32.768kHz, symbol Device:Crystal
Connections:
- net 3V3: now also J3.1 (VCC), U1.13 (VDD), U1.36 (VDD), U1.48 (VDD), C20.1, C21.1, C22.1
- net at U1.1 (DEC1): now also C11.1
- net DISP_BL: now reaches U1.12 (NFC2/P0.10)
- net DISP_RST: now reaches U1.14 (P0.11)
- net DISP_CS: now reaches U1.15 (P0.12)
- net DISP_SCLK: now reaches U1.16 (P0.13)
- net DISP_MOSI: now reaches U1.17 (P0.14)
- net DISP_DC: now reaches U1.18 (P0.15)
- net at U1.2 (P0.00/XL1): now also C15.1, Y2.1
- net at U1.21 (P0.18/SWO): now also J3.6 (SWO)
- net at U1.24 (P0.21/~{RESET}): now also J3.3 (~{RESET})
- net at U1.25 (SWDCLK): now also J3.4 (SWCLK)
- net at U1.26 (SWDIO): now also J3.2 (SWDIO)
- net at U1.3 (P0.01/XL2): now also C16.1, Y2.2
- net at U1.30 (ANT): now also L1.2
- net GND: now reaches U1.31 (VSS), U1.45 (VSS), U1.49 (VSS)
- net GND: now also J3.5 (GND), AE1.2 (Shield), C10.1, C11.2, C12.2, C13.1, C14.1, C15.2, C16.2, C17.2, C18.2, C19.2, C20.2, C21.2, C22.2, Y1.2, Y1.4
- net at U1.32 (DEC2): now also C10.2
- net at U1.33 (DEC3): now also C12.1
- net at U1.34 (XC1): now also C13.2, Y1.1
- net at U1.35 (XC2): now also C14.2, Y1.3
- net I2C_SCL: now reaches U1.38 (P0.26)
- net I2C_SDA: now reaches U1.39 (P0.27)
- net at U1.46 (DEC4): now also C18.1, L3.1
- net at U1.47 (DCC): now also L2.2
- new net: AE1.1 (A), C17.1, R16.1
- new net: C19.1, L1.1, R16.2
- new net: L2.1, L3.2
- no-connect marks 0 -> 20
Other:
- note added: "TODO: add reset button"
- moved on the sheet: J3

Commit message: fixed schematic
Parts:
- added C23: 100nF, symbol Device:C_Small
- added R17: 10k, symbol Device:R_Small
- added SW1: SW_RST, symbol Switch:SW_Push
- added TP7: TP_SCL, symbol Connector:TestPoint
- added TP8: TP_SDA, symbol Connector:TestPoint
Connections:
- net 3V3: now also R17.2
- net GND: now also C23.2
- net I2C_SCL: now also TP7.1
- net I2C_SDA: now also TP8.1
- net at J3.3 (~{RESET}), U1.24 (P0.21/~{RESET}): now also R17.1, SW1.2
- new net: C23.1, SW1.1
Other:
- note removed: "TODO: add reset button"
- moved on the sheet: J3

Commit message: changed to smd components, wip layout
Parts:
- AE1: footprint (none) -> RF_Antenna:Texas_SWRA117D_2.4GHz_Left
- C10, C11, C12, C13, C14, C15, C16, C17, C18, C19, C20, C21, C22, C23: footprint (none) -> Capacitor_SMD:C_0603_1608Metric
- L1, L2, L3: footprint (none) -> Inductor_SMD:L_0603_1608Metric
- R16, R17: footprint (none) -> Resistor_SMD:R_0603_1608Metric
- SW1: footprint (none) -> Button_Switch_SMD:SW_SPST_B3U-1000P
- TP7, TP8: footprint (none) -> TestPoint:TestPoint_Pad_D1.0mm
- Y1, Y2: footprint (none) -> Crystal:Crystal_SMD_2016-4Pin_2.0x1.6mm
Changed lines of the file:
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@@
 			)
 		)
-		(property "Footprint" ""
+		(property "Footprint" "Capacitor_SMD:C_0603_1608Metric"
 			(at 102.87 26.67 0)
 			(effects
@@
 			)
 		)
-		(property "Footprint" ""
+		(property "Footprint" "TestPoint:TestPoint_Pad_D1.0mm"
 			(at 162.56 118.11 0)
 			(effects
@@
 			)
 		)
-		(property "Footprint" ""
+		(property "Footprint" "Capacitor_SMD:C_0603_1608Metric"
 			(at 62.23 73.66 0)
 			(effects
@@
 			)
 		)
-		(property "Footprint" ""
+		(property "Footprint" "Resistor_SMD:R_0603_1608Metric"
 			(at 74.93 71.12 0)
 			(effects
@@
 			)
 		)
-		(property "Footprint" ""
+		(property "Footprint" "Capacitor_SMD:C_0603_1608Metric"
 			(at 40.64 93.98 0)
 			(effects
@@
 			)
 		)
-		(property "Footprint" ""
+		(property "Footprint" "Capacitor_SMD:C_0603_1608Metric"
 			(at 78.4352 54.61 0)
 			(effects
@@
 			)
 		)
-		(property "Footprint" ""
+		(property "Footprint" "Capacitor_SMD:C_0603_1608Metric"
 			(at 187.96 62.5348 0)
 			(effects
@@
 			)
 		)
-		(property "Footprint" ""
+		(property "Footprint" "Crystal:Crystal_SMD_2016-4Pin_2.0x1.6mm"
 			(at 87.63 92.71 0)
 			(effects
@@
 			)
 		)
-		(property "Footprint" ""
+		(property "Footprint" "TestPoint:TestPoint_Pad_D1.0mm"
 			(at 152.4 120.65 0)
 			(effects
@@
 			)
 		)
-		(property "Footprint" ""
+		(property "Footprint" "RF_Antenna:Texas_SWRA117D_2.4GHz_Left"
 			(at 53.34 60.96 0)
 			(effects
@@
 			)
 		)
-		(property "Footprint" ""
+		(property "Footprint" "Inductor_SMD:L_0603_1608Metric"
 			(at 133.35 44.45 0)
 			(effects
@@
 			)
 		)
-		(property "Footprint" ""
+		(property "Footprint" "Resistor_SMD:R_0603_1608Metric"
 			(at 40.64 74.93 0)
 			(effects
@@
 			)
 		)
-		(property "Footprint" ""
+		(property "Footprint" "Capacitor_SMD:C_0603_1608Metric"
 			(at 77.47 86.6648 0)
 			(effects
@@
 			)
 		)
-		(property "Footprint" ""
+		(property "Footprint" "Capacitor_SMD:C_0603_1608Metric"
 			(at 148.2852 41.91 0)
 			(effects
@@
 			)
 		)
-		(property "Footprint" ""
+		(property "Footprint" "Inductor_SMD:L_0603_1608Metric"
 			(at 133.35 36.83 0)
 			(effects
@@
 			)
 		)
-		(property "Footprint" ""
+		(property "Footprint" "Capacitor_SMD:C_0603_1608Metric"
 			(at 77.47 96.8248 0)
 			(effects
@@
 			)
 		)
-		(property "Footprint" ""
+		(property "Footprint" "Capacitor_SMD:C_0603_1608Metric"
 			(at 92.71 26.67 0)
 			(effects
@@
 			)
 		)
-		(property "Footprint" ""
+		(property "Footprint" "Capacitor_SMD:C_0603_1608Metric"
 			(at 85.09 73.66 0)
 			(effects
@@
 			)
 		)
-		(property "Footprint" ""
+		(property "Footprint" "Crystal:Crystal_SMD_2016-4Pin_2.0x1.6mm"
 			(at 166.37 57.15 0)
 			(effects
@@
 			)
 		)
-		(property "Footprint" ""
+		(property "Footprint" "Capacitor_SMD:C_0603_1608Metric"
 			(at 87.9348 46.99 0)
 			(effects
@@
 			)
 		)
-		(property "Footprint" ""
+		(property "Footprint" "Inductor_SMD:L_0603_1608Metric"
 			(at 96.52 71.12 0)
 			(effects
@@
 			)
 		)
-		(property "Footprint" ""
+		(property "Footprint" "Capacitor_SMD:C_0603_1608Metric"
 			(at 187.96 52.3748 0)
 			(effects
@@
 			)
 		)
-		(property "Footprint" ""
+		(property "Footprint" "Capacitor_SMD:C_0603_1608Metric"
 			(at 101.2952 54.61 0)
 			(effects
@@
 			)
 		)
-		(property "Footprint" ""
+		(property "Footprint" "Button_Switch_SMD:SW_SPST_B3U-1000P"
 			(at 35.56 85.09 0)
 			(effects
@@
 			)
 		)
-		(property "Footprint" ""
+		(property "Footprint" "Capacitor_SMD:C_0603_1608Metric"
 			(at 114.3 26.67 0)
 			(effects

Commit message: bug fix: debounce capacitor for reset button
Connections:
- net GND: now also C23.1, SW1.1; no longer C23.2
- net at J3.3 (~{RESET}), R17.1, SW1.2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: now also C23.2
Other:
- moved on the sheet: C23
Changed lines of the file:
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@@
+	)
+	(junction
+		(at 58.42 95.25)
+		(diameter 0)
+		(color 0 0 0 0)
 	)
 	(junction
@@
 	)
 	(junction
-		(at 62.23 71.12)
+		(at 40.64 95.25)
 		(diameter 0)
 		(color 0 0 0 0)
 	)
 	(junction
-		(at 50.8 107.95)
+		(at 62.23 71.12)
 		(diameter 0)
 		(color 0 0 0 0)
@@
 	)
 	(junction
+		(at 58.42 107.95)
+		(diameter 0)
+		(color 0 0 0 0)
+	)
+	(junction
 		(at 71.12 76.2)
 		(diameter 0)
@@
 	(wire
 		(pts
-			(xy 50.8 80.01) (xy 50.8 107.95)
-		)
-		(stroke
-			(width 0)
-			(type default)
-		)
-	)
-	(wire
-		(pts
 			(xy 77.47 87.63) (xy 87.63 87.63)
 		)
@@
 	(wire
 		(pts
+			(xy 40.64 95.25) (xy 40.64 97.79)
+		)
+		(stroke
+			(width 0)
+			(type default)
+		)
+	)
+	(wire
+		(pts
 			(xy 193.04 53.34) (xy 193.04 63.5)
 		)
@@
 	(wire
 		(pts
+			(xy 50.8 95.25) (xy 58.42 95.25)
+		)
+		(stroke
+			(width 0)
+			(type default)
+		)
+	)
+	(wire
+		(pts
 			(xy 62.23 76.2) (xy 71.12 76.2)
 		)
@@
 	(wire
 		(pts
+			(xy 58.42 95.25) (xy 58.42 107.95)
+		)
+		(stroke
+			(width 0)
+			(type default)
+		)
+	)
+	(wire
+		(pts
 			(xy 71.12 76.2) (xy 85.09 76.2)
 		)
@@
 	(wire
 		(pts
+			(xy 58.42 80.01) (xy 58.42 95.25)
+		)
+		(stroke
+			(width 0)
+			(type default)
+		)
+	)
+	(wire
+		(pts
 			(xy 151.13 82.55) (xy 166.37 82.55)
 		)
@@
 	(wire
 		(pts
+			(xy 40.64 90.17) (xy 40.64 95.25)
+		)
+		(stroke
+			(width 0)
+			(type default)
+		)
+	)
+	(wire
+		(pts
 			(xy 166.37 53.34) (xy 180.34 53.34)
 		)
@@
 	(wire
 		(pts
-			(xy 40.64 96.52) (xy 40.64 97.79)
-		)
-		(stroke
-			(width 0)
-			(type default)
-		)
-	)
-	(wire
-		(pts
 			(xy 123.19 30.48) (xy 147.32 30.48)
 		)
@@
 	(wire
 		(pts
-			(xy 40.64 80.01) (xy 50.8 80.01)
+			(xy 40.64 80.01) (xy 58.42 80.01)
 		)
 		(stroke
@@
 	(wire
 		(pts
-			(xy 41.91 107.95) (xy 50.8 107.95)
+			(xy 41.91 107.95) (xy 58.42 107.95)
 		)
 		(stroke
@@
 	(wire
 		(pts
-			(xy 50.8 107.95) (xy 105.41 107.95)
-		)
-		(stroke
-			(width 0)
-			(type default)
-		)
-	)
-	(wire
-		(pts
 			(xy 166.37 92.71) (xy 151.13 92.71)
 		)
@@
 	(wire
 		(pts
+			(xy 40.64 95.25) (xy 45.72 95.25)
+		)
+		(stroke
+			(width 0)
+			(type default)
+		)
+	)
+	(wire
+		(pts
 			(xy 31.75 69.85) (xy 31.75 102.87)
 		)
@@
 	(wire
 		(pts
+			(xy 58.42 107.95) (xy 105.41 107.95)
+		)
+		(stroke
+			(width 0)
+			(type default)
+		)
+	)
+	(wire
+		(pts
 			(xy 41.91 115.57) (xy 67.31 115.57)
 		)
@@
 		(pts
 			(xy 80.01 92.71) (xy 82.55 92.71)
-		)
-		(stroke
-			(width 0)
-			(type default)
-		)
-	)
-	(wire
-		(pts
-			(xy 40.64 90.17) (xy 40.64 91.44)
 		)
 		(stroke
@@
 	(symbol
 		(lib_id "Device:C_Small")
-		(at 40.64 93.98 0)
+		(at 48.26 95.25 90)
 		(unit 1)
 		(exclude_from_sim no)
@@
 		(on_board yes)
 		(dnp no)
-		(fields_autoplaced yes)
 		(property "Reference" "C23"
-			(at 43.18 92.7162 0)
-			(effects
-				(font
-					(size 1.27 1.27)
-				)
-				(justify left)
+			(at 48.26 101.346 90)
+			(effects
+				(font
+					(size 1.27 1.27)
+				)
 			)
 		)
 		(property "Value" "100nF"
-			(at 43.18 95.2562 0)
-			(effects
-				(font
-					(size 1.27 1.27)
-				)
-				(justify left)
+			(at 48.26 98.806 90)
+			(effects
+				(font
+					(size 1.27 1.27)
+				)
 			)
 		)
 		(property "Footprint" "Capacitor_SMD:C_0603_1608Metric"
-			(at 40.64 93.98 0)
+			(at 48.26 95.25 0)
 			(effects
 				(font
@@
 		)
 		(property "Datasheet" "~"
-			(at 40.64 93.98 0)
+			(at 48.26 95.25 0)
 			(effects
 				(font
@@
 		)
 		(property "Description" "Unpolarized capacitor, small symbol"
-			(at 40.64 93.98 0)
-			(effects
-				(font
+			(at 48.26 95.25 0)
+			(effects
+				(font

Commit message: fixed antenna layout
wip: placing components
Parts:
- removed AE1: BLE, RF_Antenna:Texas_SWRA117D_2.4GHz_Left, symbol Device:Antenna_Shield
- added AE1: ~, RF_Antenna:Antenna_BLE, symbol RF_Bluetooth:PCB_Antenna_BLE_Custom
- added C25: 0.8pF, Capacitor_SMD:C_0201_0603Metric, symbol Device:C_Small
- added C26: NC, Capacitor_SMD:C_0201_0603Metric, symbol Device:C_Small
- C17: value 0.8pF -> 1.5pF; footprint Capacitor_SMD:C_0603_1608Metric -> Capacitor_SMD:C_0201_0603Metric
- C19: value 0.8pF -> 0.5pF; footprint Capacitor_SMD:C_0603_1608Metric -> Capacitor_SMD:C_0201_0603Metric
- L1: value 3.9nH -> 4.7nH; footprint Inductor_SMD:L_0603_1608Metric -> Inductor_SMD:L_0201_0603Metric
- R16: footprint Resistor_SMD:R_0603_1608Metric -> Resistor_SMD:R_0201_0603Metric
- Y2: footprint Crystal:Crystal_SMD_2016-4Pin_2.0x1.6mm -> Crystal:Crystal_SMD_3215-2Pin_3.2x1.5mm
Connections:
- net GND: now also C25.2, C26.2
- net at L1.2, U1.30 (ANT): now also C25.1
- net at C17.1, R16.1: now also AE1.1 (FEED)
- net at C19.1, L1.1, R16.2: now also C26.1
Other:
- moved on the sheet: C17, C19, L1, R16

Commit message: Added name and revision
Other:
- title: (none) -> air-ctrl
Changed lines of the file:
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@@
 	(generator_version "9.0")
 	(paper "A4")
+	(title_block
+		(title "air-ctrl")
+		(date "2025-10-18")
+		(rev "1.1")
+	)
 	(junction
 		(at 87.63 97.79)

Commit message: Fixed some R and C values, added missing 3D models
Parts:
- C20, C21: value 100uF -> 0.1uF
Changed lines of the file:
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@@
 			)
 		)
-		(property "Value" "100uF"
+		(property "Value" "0.1uF"
 			(at 105.41 27.9462 0)
 			(effects
@@
 			)
 		)
-		(property "Value" "100uF"
+		(property "Value" "0.1uF"
 			(at 95.25 27.9462 0)
 			(effects
