File: hardware/mcu.kicad_sch (KiCad schematic)
At the start: 29 parts, among them J3 Conn_ARM_SWD_TagConnect_TC203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, SW1 SW_RST, U1 nRF52832-QFxx, Y1 32MHz, Y2 32.768kHz

Commit message: Exclude Test points and such from BOM
Parts:
- AE1, C26, TP7, TP8: now left out of the parts list
Changed lines of the file:
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@@
 		(unit 1)
 		(exclude_from_sim no)
-		(in_bom yes)
+		(in_bom no)
 		(on_board yes)
 		(dnp no)
@@
 		(unit 1)
 		(exclude_from_sim no)
-		(in_bom yes)
+		(in_bom no)
 		(on_board yes)
 		(dnp no)
@@
 		(unit 1)
 		(exclude_from_sim no)
-		(in_bom yes)
+		(in_bom no)
 		(on_board yes)
 		(dnp no)
@@
 		(unit 1)
 		(exclude_from_sim no)
-		(in_bom yes)
-		(on_board yes)
-		(dnp no)
+		(in_bom no)
+		(on_board yes)
+		(dnp no)

Commit message: Fixes after nordic review
ready to order!
Parts:
- removed C10: 100nF, Capacitor_SMD:C_0603_1608Metric, symbol Device:C
- removed C19: 0.5pF, Capacitor_SMD:C_0201_0603Metric, symbol Device:C_Small
- L1: value 4.7nH -> 3.9nH
Connections:
- no-connect marks 20 -> 21
Other:
- moved on the sheet: C12
